File: Hardware/Plazma_Circuit/Plazma_Circuit.sch (KiCad schematic (older format))
At the start: 61 parts, among them J1 Screw_Terminal_01x02, J10 Y2 Axis, J11 X Axis, J2 R Axis, J3 DISPLAY, J4 STOPS, J5 V to FREQ, J6 TORCH, J7 SPARE, J8 Z Axis, J9 Y1Axis, K1 TOARCH TRIGGER, U1 MC1413, U2 ESP32Master, U3 ESP32 Torch, U4 MC1413, U5 MC1413

Commit message: Add Existing Kicad Files, Add BDRING, Start new schematic
Parts:
- K1: value TOARCH TRIGGER -> TORCH TRIGGER
- PS1, PS2: symbol Plazma:DC-DC_BuckAdg -> Plazma_Circuit-rescue:DC-DC_BuckAdg-Plazma
- U2, U3: symbol Plazma:ESP32DevkitV1 -> Plazma_Circuit-rescue:ESP32DevkitV1-Plazma
Changed lines of the file:
@@
 $EndComp
 $Comp
-L Plazma:DC-DC_BuckAdg PS2
+L Plazma_Circuit-rescue:DC-DC_BuckAdg-Plazma PS2
 U 1 1 5FDBFD38
 P 2200 5850
@@
 $EndComp
 $Comp
-L Plazma:ESP32DevkitV1 U2
+L Plazma_Circuit-rescue:ESP32DevkitV1-Plazma U2
 U 1 1 5FDD0ECB
 P 4200 3450
@@
 $EndComp
 $Comp
-L Plazma:ESP32DevkitV1 U3
+L Plazma_Circuit-rescue:ESP32DevkitV1-Plazma U3
 U 1 1 5FDD0D96
 P 5600 3450
@@
 $EndComp
 $Comp
-L Plazma:DC-DC_BuckAdg PS1
+L Plazma_Circuit-rescue:DC-DC_BuckAdg-Plazma PS1
 U 1 1 5FDD74AE
 P 2200 4650
@@
 P 8200 5700
 F 0 "K1" V 7633 5700 50  0000 C CNN
-F 1 "TOARCH TRIGGER" V 7724 5700 50  0000 C CNN
+F 1 "TORCH TRIGGER" V 7724 5700 50  0000 C CNN
 F 2 "Relay_THT:Relay_DPDT_Omron_G5V-2" H 9340 5660 50  0001 C CNN
 F 3 "https://www.finder-relais.net/de/finder-relais-serie-40.pdf" H 8200 5700 50  0001 C CNN
