File: Hardware/Dring Heath Small/_autosave-BDringController.sch (KiCad schematic (older format))
At the start: 94 parts, among them J1 Module 1, J10 Module 3, J11 JTAG, J12 Shift Regs and Motor Drvs, J13 Module 4, J14 Module 5, J15 Micro_SD_Card, J16 Pin, J17 Pin, J18 Pin, J19 Pin, J2 Jumper, J20 Pin, J21 Pin, J22 AUX GPIO, J3 Motor, J4 Module 1, J5 Ext Mot Drv, J6 01x02, J7 THC_Display, J8 Module 2, J9 VMot, U1 ESP32_38p, U10 Y, U11 z, U12 A, U13 B, U14 C, U2 74LVC157A, U3 ESP32_38p, U4 TC1262-33, U5 74AHCT595, U6 74AHCT595, U7 74AHCT595, U8 74AHCT595, U9 X

Commit message: more routing and added Dring large folder
Connections:
- net A_CS: now also U7.7 (QH)
- net A_Dir: now also U7.5 (QF); no longer U7.6 (QG)
- net A_Enable: now also U7.4 (QE); no longer U7.5 (QF)
- net A_Step: now also U7.6 (QG); no longer U7.7 (QH)
- net GND: now also J6.2 (Pin_2), PS1.2 (-Vin), PS2.2 (-Vin), U7.13 (~OE), U7.8 (GND)
- net GrbZDir: now also U7.1 (QB); no longer U7.2 (QC)
- net GrbZEn: now also U7.15 (QA); no longer U7.1 (QB)
- net GrbZStep: now also U7.2 (QC); no longer U7.3 (QD)
- net I2S_BCK: now also U7.11 (SRCLK); no longer U7.10 (~SRCLR)
- net I2S_WS: now also U7.12 (RCLK); no longer U7.13 (~OE)
- net VCC: now also U7.10 (~SRCLR)
- net Z_CS: now also U7.3 (QD); no longer U7.4 (QE)
- net at U5.9 (QH'): now also U7.14 (SER)
- net at U7.9 (QH'): now also U6.14 (SER)
Other:
- moved on the sheet: U7
Changed lines of the file:
@@
 L 74xx:74AHCT595 U7
 U 1 1 5FE6B667
-P 11650 2550
-F 0 "U7" H 11650 2350 50  0000 C CNN
-F 1 "74AHCT595" H 11600 2200 50  0000 C CNN
-F 2 "Package_SO:SO-16_5.3x10.2mm_P1.27mm" H 11650 2550 50  0001 C CNN
-F 3 "https://assets.nexperia.com/documents/data-sheet/74AHC_AHCT595.pdf" H 11650 2550 50  0001 C CNN
-	1    11650 2550
+P 11650 2650
+F 0 "U7" H 11650 2450 50  0000 C CNN
+F 1 "74AHCT595" H 11600 2300 50  0000 C CNN
+F 2 "Package_SO:SO-16_5.3x10.2mm_P1.27mm" H 11650 2650 50  0001 C CNN
+F 3 "https://assets.nexperia.com/documents/data-sheet/74AHC_AHCT595.pdf" H 11650 2650 50  0001 C CNN
+	1    11650 2650
 	1    0    0    -1
 $EndComp
@@
 $EndComp
 Wire Wire Line
-	11250 2750 11250 3250
-Wire Wire Line
 	11250 3350 11650 3350
 Wire Wire Line
@@
 	-1   0    0    1
 $EndComp
-Connection ~ 11250 2750
 $Comp
 L Device:C_Small C25
@@
 Wire Wire Line
 	5900 1400 6050 1400
+Connection ~ 6050 1400
+Connection ~ 11650 3350
+Wire Wire Line
+	11250 2850 11250 3350
+$Comp
+L power:GND #PWR0106
+U 1 1 605E21DB
+P 6250 7100
+F 0 "#PWR0106" H 6250 6850 50  0001 C CNN
+F 1 "GND" H 6255 6927 50  0000 C CNN
+F 2 "" H 6250 7100 50  0001 C CNN
+F 3 "" H 6250 7100 50  0001 C CNN
+	1    6250 7100
+	1    0    0    -1
+$EndComp
+Wire Wire Line
+	6100 7100 6250 7100
 Wire Bus Line
 	9500 1650 9500 5450
-Connection ~ 6050 1400
 $EndSCHEMATC
