File: Hardware/Dring Heath Small/Torch Module/Torch Module.sch (KiCad schematic (older format))
At the start: 75 parts, among them J1 Torch, J10 Module conn, J11 Conn_01x18_Male, J12 Conn_01x02_Male, J13 Conn_01x02_Male, J14 Conn_01x02_Male, J15 Module conn, J2 Module3, J3 Conn_01x18_Male, J4 Limit, J6 Motor, J7 Module1, J8 Torch, J9 2.54 pin, K1 G6E, Q1 IRLML2402, Q2 IRLML2402, Q3 IRLML2402, Q4 IRLML2402, Q5 IRLML2402, U1 ULN2002, U2 NCV8114ASN150T1G, U3 ADS1115IDGS

Commit message: routed a/d board
put simulation on excel bom
Parts:
- removed J13: Conn_01x02_Male, Connector_PinHeader_2.54mm:PinHeader_1x02_P2.54mm_Vertical, symbol Connector:Conn_01x02_Male
- added J13: ~, Connector_PinHeader_2.54mm:PinHeader_2x02_P2.54mm_Vertical, symbol Connector_Generic:Conn_02x02_Odd_Even
Connections:
- net at C1.1, C2.1, J1.10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: now also J13.4 (Pin_4)
- net at J1.3: now also J13.3 (Pin_3)
- net at J1.4: now also J13.1 (Pin_1); no longer R3.1
- net at C6.2, C7.2, D2.2 (A)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: no longer U3.6 (AIN2), U3.7 (AIN3)
- new net: J13.2 (Pin_2), R3.1
- no-connect marks 44 -> 46
Changed lines of the file:
@@
 	3650 1000 3650 1500
 Wire Wire Line
-	2650 1850 2650 1350
-Wire Wire Line
-	2400 1850 2650 1850
+	2400 1850 2550 1850
 Wire Wire Line
 	2400 2150 2400 1850
@@
 Wire Wire Line
 	2450 1900 2450 2050
-Wire Wire Line
-	2850 1900 2450 1900
-Wire Wire Line
-	2850 1800 2850 1900
-Wire Wire Line
-	2850 1800 2900 1800
 Connection ~ 3650 1900
 Wire Wire Line
@@
 AR Path="/61A6728B" Ref="R1"  Part="1"
 AR Path="/61469ABE/61A6728B" Ref="R?"  Part="1"
-F 0 "R1" V 2195 1500 50  0000 C CNN
-F 1 "3.3K" V 2286 1500 50  0000 C CNN
+F 0 "R1" V 2500 1300 50  0000 C CNN
+F 1 "3.3K" V 2500 1450 50  0000 C CNN
 F 2 "Resistor_SMD:R_0603_1608Metric_Pad0.98x0.95mm_HandSolder" V 2440 1490 50  0001 C CNN
 F 3 "~" H 2400 1500 50  0001 C CNN
@@
 AR Path="/61A67257" Ref="R4"  Part="1"
 AR Path="/61469ABE/61A67257" Ref="R?"  Part="1"
-F 0 "R4" V 2895 1500 50  0000 C CNN
+F 0 "R4" V 3200 1500 50  0000 C CNN
 F 1 "10k" V 2986 1500 50  0000 C CNN
 F 2 "Resistor_SMD:R_0603_1608Metric_Pad0.98x0.95mm_HandSolder" V 3140 1490 50  0001 C CNN
@@
 AR Path="/61A6724B" Ref="R3"  Part="1"
 AR Path="/61469ABE/61A6724B" Ref="R?"  Part="1"
-F 0 "R3" H 3100 1750 50  0000 R CNN
-F 1 "3.3K" H 3100 1600 50  0000 R CNN
+F 0 "R3" H 2850 1700 50  0000 R CNN
+F 1 "3.3K" H 2900 1800 50  0000 R CNN
 F 2 "Resistor_SMD:R_0603_1608Metric_Pad0.98x0.95mm_HandSolder" V 2940 1640 50  0001 C CNN
 F 3 "~" H 2900 1650 50  0001 C CNN
@@
 IO 21recieve handover
 Wire Wire Line
-	2650 1000 1900 1000
-Wire Wire Line
 	1900 1000 1900 1450
 Wire Wire Line
@@
 $EndComp
 NoConn ~ 4850 1850
-Wire Wire Line
-	2650 1000 2900 1000
-Connection ~ 2650 1000
 Connection ~ 3250 1000
 Wire Wire Line
@@
 U 1 1 60201FC2
 P 2900 1350
-F 0 "RV1" H 2833 1396 50  0000 R CNN
-F 1 "2K" H 2833 1305 50  0000 R CNN
+F 0 "RV1" H 2850 1500 50  0000 R CNN
+F 1 "2K" H 2850 1400 50  0000 R CNN
 F 2 "Potentiometer_THT:Potentiometer_Bourns_3339S_Horizontal" H 2900 1350 50  0001 C CNN
 F 3 "~" H 2900 1350 50  0001 C CNN
@@
 $EndComp
 $Comp
-L Connector:Conn_01x02_Male J13
-U 1 1 60313235
-P 2450 1250
-F 0 "J13" H 2558 1431 50  0000 C CNN
-F 1 "Conn_01x02_Male" H 2558 1340 50  0000 C CNN
-F 2 "Connector_PinHeader_2.54mm:PinHeader_1x02_P2.54mm_Vertical" H 2450 1250 50  0001 C CNN
-F 3 "~" H 2450 1250 50  0001 C CNN
-	1    2450 1250
-	1    0    0    -1
-$EndComp
-Wire Wire Line
-	2650 1250 2650 1000
-$Comp
 L Connector:Conn_01x02_Male J14
 U 1 1 60313D52
@@
 Wire Wire Line
 	4000 5900 4100 5900
-Wire Wire Line
-	4100 6000 4100 6100
-Wire Wire Line
-	4100 6400 4500 6400
-Connection ~ 4100 6100
 Connection ~ 4500 6400
 Wire Wire Line
@@
 Wire Wire Line
 	2450 5800 2450 5900
-Wire Wire Line
-	4100 6100 4100 6400
 Connection ~ 4500 5400
 Wire Wire Line
@@
 	3350 6200 3350 6400
 Wire Wire Line
-	3350 6400 4100 6400
-Connection ~ 4100 6400
-Wire Wire Line
 	6350 5100 6350 6200
 Wire Wire Line
@@
 NoConn ~ 8450 4350
 NoConn ~ 8550 4350
+$Comp
+L Connector_Generic:Conn_02x02_Odd_Even J13
+U 1 1 60218639
+P 2650 1650
+F 0 "J13" V 2700 1700 50  0000 L CNN
+F 1 "~" V 3250 700 50  0000 L CNN
+F 2 "Connector_PinHeader_2.54mm:PinHeader_2x02_P2.54mm_Vertical" H 2650 1650 50  0001 C CNN
+F 3 "~" H 2650 1650 50  0001 C CNN
+	1    2650 1650
+	0    1    -1   0
+$EndComp
+Wire Wire Line
+	2800 1800 2800 1350
+Wire Wire Line
+	2800 1350 2650 1350
+Wire Wire Line
+	2800 1800 2900 1800
+Wire Wire Line
+	2550 1350 2550 1000
+Connection ~ 2550 1000
+Wire Wire Line
+	2550 1000 1900 1000
+Wire Wire Line
+	2450 1900 2650 1900
+Wire Wire Line
+	2650 1900 2650 1850
+Wire Wire Line
+	2550 1000 2900 1000
+Wire Wire Line
+	3350 6400 4500 6400
+NoConn ~ 4100 6000
+NoConn ~ 4100 6100
 $EndSCHEMATC
