File: Hardware/Main Board/BDringController.kicad_pcb (KiCad board)
At the start: 2 copper layers, 144.8 x 131.4 mm, 98 parts, among them J1 AUX GPIO, J10 Module 2, J11 VMot, J12 Module 3, J13 Shift Regs and Motor Drvs, J14 Module 4, J15 Module 5, J16 Micro_SD_Card, J17 Pin, J18 Pin, J19 Pin, J20 Pin, J21 Pin, J22 Pin, J23 RST, J24 RST, J3 Torch module, J4 Jumper, J5 Motor, J6 Module 1, J7 Ext Mot Drv, J8 01x02, J9 THC_Display, U1 ESP32_38p, U10 Y, U11 z, U12 A, U13 B, U14 C, U2 74LVC157A, U3 ESP32_38p, U4 BL8071CLATR33, U5 74AHCT595, U6 74AHCT595, U7 74AHCT595, U8 74AHCT595, U9 X

Commit message: Gerbers for Main Board, minimal DRC errors
Parts:
- J9: footprint Modules:RJ45_BEL_SS74301-00x_Vertical -> Connector_RJ:RJ45_OST_PJ012-8P8CX_Vertical
- U1, U3: footprint Modules:ESP32_38p -> Libraries - Plasma-Board:ESP32_38p
- moved C25 3.51 mm to (196.5, 123.8)
- moved J9 2.31 mm to (122.2, 49.2)
- moved H9 0.45 mm to (116.4, 78.3), turned to 90 degrees
Connections:
- H10 pad 1: Net-(H10-Pad1) -> +15V
- H9 pad 1: Net-(H9-Pad1) -> Net-(H8-Pad1)
- J1 pad 5: Net-(J1-Pad5) -> (no net)
- J1 pad 6: Net-(J1-Pad6) -> (no net)
- J16 pad 1: Net-(J16-Pad1) -> (no net)
- J16 pad 8: Net-(J16-Pad8) -> (no net)
- J8 pad 1: Net-(H9-Pad1) -> Net-(H8-Pad1)
- PS1 pad 1: Net-(H9-Pad1) -> Net-(H8-Pad1)
- PS2 pad 1: Net-(H9-Pad1) -> Net-(H8-Pad1)
- U1 pad 1: Net-(U1-Pad1) -> (no net)
- U1 pad 10: Net-(U1-Pad10) -> (no net)
- U1 pad 2: Net-(U1-Pad2) -> (no net)
- U1 pad 20: Net-(U1-Pad20) -> (no net)
- U1 pad 23: Net-(U1-Pad23) -> (no net)
- U1 pad 24: Net-(U1-Pad24) -> (no net)
- U1 pad 3: Net-(U1-Pad3) -> (no net)
- U1 pad 34: Net-(U1-Pad34) -> (no net)
- U1 pad 35: Net-(U1-Pad35) -> (no net)
- U1 pad 36: Net-(U1-Pad36) -> (no net)
- U1 pad 37: Net-(U1-Pad37) -> (no net)
- U1 pad 4: Net-(U1-Pad4) -> (no net)
- U1 pad 5: Net-(U1-Pad5) -> (no net)
- U1 pad 6: Net-(U1-Pad6) -> (no net)
- U1 pad 7: Net-(U1-Pad7) -> (no net)
- U10 pad 18: Net-(U10-Pad18) -> (no net)
- U13 pad 18: Net-(U13-Pad18) -> (no net)
- U14 pad 18: Net-(U14-Pad18) -> (no net)
- U2 pad 12: Net-(U2-Pad12) -> (no net)
- U2 pad 13: Net-(U2-Pad13) -> (no net)
- U2 pad 14: Net-(U2-Pad14) -> (no net)
- U3 pad 1: Net-(U3-Pad1) -> (no net)
- U3 pad 15: Net-(U3-Pad15) -> (no net)
- U3 pad 16: Net-(U3-Pad16) -> (no net)
- U3 pad 2: Net-(U3-Pad2) -> (no net)
- U3 pad 20: Net-(U3-Pad20) -> (no net)
- U3 pad 3: Net-(U3-Pad3) -> (no net)
- U3 pad 35: Net-(U3-Pad35) -> (no net)
- U3 pad 36: Net-(U3-Pad36) -> (no net)
- U3 pad 37: Net-(U3-Pad37) -> (no net)
- U3 pad 6: Net-(U3-Pad6) -> (no net)
- U8 pad 4: Net-(U8-Pad4) -> (no net)
- U8 pad 5: Net-(U8-Pad5) -> (no net)
- U8 pad 6: Net-(U8-Pad6) -> (no net)
- U8 pad 7: Net-(U8-Pad7) -> (no net)
- U8 pad 9: Net-(U8-Pad9) -> (no net)
- U9 pad 18: Net-(U9-Pad18) -> (no net)
Routing:
- net GND: track 706.9 -> 754.2 mm, vias 50 -> 48
- net Net-(H8-Pad1): track 0.00 -> 39.8 mm
- net Net-(H9-Pad1): track 35.0 -> 0.00 mm
- net +5V: track 154.5 -> 148.7 mm
- net C_Limit: track 95.2 -> 91.7 mm
- net B_Limit: track 95.5 -> 92.1 mm
- net +3V3: track 185.8 -> 189.1 mm
- net Net-(J9-Pad4): track 33.9 -> 30.7 mm
- net Net-(J9-Pad7): track 66.8 -> 63.6 mm
- net Net-(J9-Pad3): track 34.3 -> 31.1 mm
- net A_Dir: track 38.0 -> 35.7 mm
- net X_CS: track 36.0 -> 33.7 mm
- net Net-(J22-Pad4): track 23.4 -> 22.1 mm
- net Net-(J22-Pad2): track 27.2 -> 25.9 mm
- net GPIO27: track 97.8 -> 96.7 mm
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