File: Hardware/Main Board/BDringController.sch (KiCad schematic (older format))
At the start: 98 parts, among them J1 AUX GPIO, J10 Module 2, J11 VMot, J12 Module 3, J13 Shift Regs and Motor Drvs, J14 Module 4, J15 Module 5, J16 Micro_SD_Card, J17 Pin, J18 Pin, J19 Pin, J20 Pin, J21 Pin, J22 Pin, J23 RST, J24 RST, J3 Torch module, J4 Jumper, J5 Motor, J6 Module 1, J7 Ext Mot Drv, J8 01x02, J9 THC_Display, U1 ESP32_38p, U10 Y, U11 z, U12 A, U13 B, U14 C, U2 74LVC157A, U3 ESP32_38p, U4 BL8071CLATR33, U5 74AHCT595, U6 74AHCT595, U7 74AHCT595, U8 74AHCT595, U9 X

Commit message: Gerbers for Main Board, minimal DRC errors
Parts:
- J9: footprint Modules:RJ45_BEL_SS74301-00x_Vertical -> Connector_RJ:RJ45_OST_PJ012-8P8CX_Vertical
- U1, U3: footprint Modules:ESP32_38p -> Libraries - Plasma-Board:ESP32_38p; symbol BDringController-rescue:ESP32_38p-My_Library -> My_Library:ESP32_38p
Changed lines of the file:
@@
 $EndComp
 $Comp
-L BDringController-rescue:ESP32_38p-My_Library U3
+L My_Library:ESP32_38p U3
 U 1 1 5FF3DD1B
 P 8050 3250
 F 0 "U3" V 9515 3300 50  0000 C CNN
 F 1 "ESP32_38p" V 9424 3300 50  0000 C CNN
-F 2 "Modules:ESP32_38p" H 8050 3250 50  0001 C CNN
+F 2 "Libraries - Plasma-Board:ESP32_38p" H 8050 3250 50  0001 C CNN
 F 3 "" H 8050 3250 50  0001 C CNN
 	1    8050 3250
@@
 GRBL ESP32
 $Comp
-L BDringController-rescue:ESP32_38p-My_Library U1
+L My_Library:ESP32_38p U1
 U 1 1 60718252
 P 4450 2500
 F 0 "U1" V 5915 2550 50  0000 C CNN
 F 1 "ESP32_38p" V 5824 2550 50  0000 C CNN
-F 2 "Modules:ESP32_38p" H 4450 2500 50  0001 C CNN
+F 2 "Libraries - Plasma-Board:ESP32_38p" H 4450 2500 50  0001 C CNN
 F 3 "" H 4450 2500 50  0001 C CNN
 	1    4450 2500
@@
 F 0 "J9" H 6257 4067 50  0000 C CNN
 F 1 "THC_Display" H 6257 3976 50  0000 C CNN
-F 2 "Modules:RJ45_BEL_SS74301-00x_Vertical" V 6200 3425 50  0001 C CNN
+F 2 "Connector_RJ:RJ45_OST_PJ012-8P8CX_Vertical" V 6200 3425 50  0001 C CNN
 F 3 "~" V 6200 3425 50  0001 C CNN
 	1    6200 3400
@@
 	6500 6200 6500 6150
 Connection ~ 6500 6150
-$Comp
-L power:+5V #PWR0101
-U 1 1 6072477D
-P 2600 4000
-F 0 "#PWR0101" H 2600 3850 50  0001 C CNN
-F 1 "+5V" H 2615 4173 50  0000 C CNN
-F 2 "" H 2600 4000 50  0001 C CNN
-F 3 "" H 2600 4000 50  0001 C CNN
-	1    2600 4000
-	1    0    0    -1
-$EndComp
 Wire Wire Line
 	5400 3200 5400 3800
@@
 Wire Wire Line
 	6350 6150 6400 6150
-Wire Bus Line
-	9500 1650 9500 5450
 Connection ~ 6400 6150
 Wire Wire Line
 	6400 6150 6400 6100
+Wire Bus Line
+	9500 1650 9500 5450
 $EndSCHEMATC

Commit message: Ordered parts, finished modules, fixed rj45
Parts:
- C1, C10, C11, C12, C13, C15, C17, C19, C2, C21, C23, C25, C5, C6, C7: LCSC (none) -> C107569; Part Number (none) -> 0603B104M250CT
- C14, C16, C18, C20, C22, C24, C3, C4: LCSC (none) -> C250026; Part Number (none) -> OCV331M1DTR-1013
- C9: LCSC (none) -> C344022; Part Number (none) -> GRM188R61E106KA73D
- D1: LCSC (none) -> C189958; Part Number (none) -> MSCD104H
- D2, D3, D4, D5: LCSC (none) -> C84263; Part Number (none) -> NCD0603R1
- J10, J12, J14, J15, J3, J6: symbol BDringController-rescue:IO_connector-My_Library -> BDringController-rescue:IO_connector-My_Library-BDringController-rescue
- J16: LCSC (none) -> C114218; Part Number (none) -> DM3AT-SF-PEJM5
- J7, J8: LCSC (none) -> C415432; Part Number (none) -> JL124D-35002G01
- L1, L2: LCSC (none) -> C439349; Part Number (none) -> GCNR4030-220MC
- PS1, PS2: symbol BDringController-rescue:DC-DC_BuckAdg-My_Library -> BDringController-rescue:DC-DC_BuckAdg-My_Library-BDringController-rescue
- R1, R10, R11, R12, R2, R3, R4, R9: LCSC (none) -> C22548
- R5, R6, R7, R8: LCSC (none) -> C144081
- U1, U3: symbol My_Library:ESP32_38p -> BDringController-rescue:ESP32_38p-My_Library
- U10, U11, U12, U13, U14, U9: symbol BDringController-rescue:Motor_driver-My_Library -> BDringController-rescue:Motor_driver-My_Library-BDringController-rescue
- U2: symbol BDringController-rescue:74LVC157A-My_Library -> BDringController-rescue:74LVC157A-My_Library-BDringController-rescue; LCSC (none) -> C707097; Part Number (none) -> XL74LS157
- U4: LCSC (none) -> C401677; Part Number (none) -> BL8071CLATR33
- U5, U6, U7, U8: LCSC (none) -> C503428; Part Number (none) -> 74AHCT595D,118
