File: Hardware/Torch Module/Torch Module.sch (KiCad schematic (older format))
At the start: 82 parts, among them J1 Torch, J10 Module conn, J11 Conn_01x18_Male, J12 Conn_01x02_Male, J14 Conn_01x02_Male, J15 Module conn, J16 Reset, J17 Reset, J18 Reset, J2 Module3, J3 Conn_01x18_Male, J4 Limit, J6 8P8C_LED_Shielded, J7 Module1, J8 Torch, J9 2.54 pin, K1 G6E, Q1 IRLML2402, Q2 IRLML2402, Q3 IRLML2402, Q4 IRLML2402, Q5 IRLML2402, U1 ULN2002, U2 NCV8114ASN150T1G, U3 ADS1115IDGS

Commit message: fix all erc and drc, add lcsc pns, fix rj45, fix footprints
Parts:
- C1, C7: LCSC (none) -> C1591; PN (none) -> CL10B104KB8NNNC
- C2, C4, C5, C6, C8: LCSC (none) -> C29936; PN (none) -> CL10B105KA8NNNC
- C3: LCSC (none) -> C21122; PN (none) -> CL10B223KB8NNNC
- D1: LCSC (none) -> C426570; PN (none) -> SM4007PL A7
- D2, D3: LCSC (none) -> C189958; PN (none) -> MSCD104H
- FB1: LCSC (none) -> C82155; PN (none) -> BLM18HE152SN1D
- FB2: value ~ -> BLM18HE152SN1D; LCSC (none) -> C82155; PN (none) -> BLM18HE152SN1D
- J1, J4, J8: footprint Modules:RJ45_Torb_Vertical -> Connector_RJ:RJ45_BEL_SS74301-00x_Vertical; symbol My_library:8P8C_Shielded -> 8P8C_Shielded:8P8C_Shielded; LCSC (none) -> C179768; PN (none) -> 51F-1210GY2D2NL
- J11, J3: footprint Modules:ClearpathDriver -> Libraries - Plasma-Board:ClearpathDriver
- J6: symbol My_library:8P8C_LED_Shielded -> Torch_Module-cache:My_library_8P8C_LED_Shielded; LCSC (none) -> C133529; PN (none) -> C133529
- K1: LCSC (none) -> C469134; PN (none) -> G6E-134P-ST-US-DC12
- Q1, Q2, Q3, Q4, Q5: LCSC (none) -> C2588; PN (none) -> IRLML2402TRPBF
- R1, R3: LCSC (none) -> C144661; PN (none) -> AC0603FR-073K3L
- R10, R18, R20, R22, R23, R24, R25, R26, R27, R28, R29, R38, R39, R6, R7, R8: LCSC (none) -> C125935; PN (none) -> AC0603FR-07200RL
- R11, R12: value 3.3k -> 3.3K; LCSC (none) -> C144661; PN (none) -> AC0603FR-073K3L
- R13, R14, R2, R30, R32, R33, R40, R41: value 1k -> 1K; LCSC (none) -> C22548; PN (none) -> RC0603FR-071KL
- R15, R16, R17, R19, R21, R4, R5, R9: value 10k -> 10K; LCSC (none) -> C144081; PN (none) -> AF0603FR-0710KL
- R31: value 2k -> 2K; LCSC (none) -> C125933; PN (none) -> AC0603FR-072KL
- R34, R35, R36, R37: LCSC (none) -> C144674; PN (none) -> AC0603FR-072K4L
- U1: LCSC (none) -> C91899; PN (none) -> ULN2002D1013TR
- U2: LCSC (none) -> C256532; PN (none) -> NCV8114ASN150T1G
- U3: LCSC (none) -> C37593; PN (none) -> ADS1115IDGSR
Connections:
- wire segments 361 -> 360

Commit message: Ordered parts, finished modules, fixed rj45
Parts:
- added H1, H2: MountingHole, MountingHole:MountingHole_3.2mm_M3, symbol Mechanical:MountingHole
- J1, J4, J8: footprint Connector_RJ:RJ45_BEL_SS74301-00x_Vertical -> RJHSE-3380:RJHSE3384; symbol 8P8C_Shielded:8P8C_Shielded -> 8P8C_Shielded:8P8C_Shielded_Custom
Connections:
- net at C4.1, C5.1, J7.1 (Pin_1)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: now also J4.10, J4.11, J4.12, J4.9, J4.MH1, J4.MH2; no longer J4.SH
- net at C1.1, C2.1, J13.3 (Pin_3)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: now also J1.10, J1.11, J1.12, J1.9, J1.MH1, J1.MH2; no longer J1.SH
- net at J10.1 (Pin_1), J10.12 (Pin_12), J16.2 (Pin_2)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: now also J8.10, J8.11, J8.12, J8.9, J8.MH1, J8.MH2; no longer J8.SH
Changed lines of the file:
@@
 	3950 2450 4350 2450
 Connection ~ 4350 2450
-$Comp
-L 8P8C_Shielded:8P8C_Shielded J4
-U 1 1 600B48EF
-P 8150 1550
-F 0 "J4" H 7950 2100 50  0000 R CNN
-F 1 "Limit" H 8000 2200 50  0000 R CNN
-F 2 "Connector_RJ:RJ45_BEL_SS74301-00x_Vertical" V 8150 1575 50  0001 C CNN
-F 3 "https://datasheet.lcsc.com/szlcsc/1811141123_Shanghai-YDS-Tech-51F-1210GY2D2NL_C179768.pdf" V 8150 1575 50  0001 C CNN
-F 4 "C179768" H 8150 1550 50  0001 C CNN "LCSC"
-F 5 "51F-1210GY2D2NL" H 8150 1550 50  0001 C CNN "PN"
-	1    8150 1550
-	1    0    0    -1
-$EndComp
 Wire Wire Line
 	8150 950  8700 950
@@
 	-1   0    0    1
 $EndComp
-$Comp
-L 8P8C_Shielded:8P8C_Shielded J1
-U 1 1 600A1FE7
-P 1900 2050
-F 0 "J1" H 1700 2600 50  0000 R CNN
-F 1 "Torch" H 1750 2700 50  0000 R CNN
-F 2 "Connector_RJ:RJ45_BEL_SS74301-00x_Vertical" V 1900 2075 50  0001 C CNN
-F 3 "https://datasheet.lcsc.com/szlcsc/1811141123_Shanghai-YDS-Tech-51F-1210GY2D2NL_C179768.pdf" V 1900 2075 50  0001 C CNN
-F 4 "C179768" H 1900 2050 50  0001 C CNN "LCSC"
-F 5 "51F-1210GY2D2NL" H 1900 2050 50  0001 C CNN "PN"
-	1    1900 2050
-	1    0    0    -1
-$EndComp
 Wire Wire Line
 	2300 2350 2500 2350
@@
 Wire Wire Line
 	3050 1000 3250 1000
-$Comp
-L 8P8C_Shielded:8P8C_Shielded J8
-U 1 1 6023A990
-P 5800 4250
-F 0 "J8" H 5600 4800 50  0000 R CNN
-F 1 "Torch" H 5650 4900 50  0000 R CNN
-F 2 "Connector_RJ:RJ45_BEL_SS74301-00x_Vertical" V 5800 4275 50  0001 C CNN
-F 3 "https://datasheet.lcsc.com/szlcsc/1811141123_Shanghai-YDS-Tech-51F-1210GY2D2NL_C179768.pdf" V 5800 4275 50  0001 C CNN
-F 4 "C179768" H 5800 4250 50  0001 C CNN "LCSC"
-F 5 "51F-1210GY2D2NL" H 5800 4250 50  0001 C CNN "PN"
-	1    5800 4250
-	0    1    -1   0
-$EndComp
 Wire Wire Line
 	5500 3150 5500 3250
@@
 	6400 3850 6400 4150
 Connection ~ 6400 4150
-Wire Wire Line
-	5300 4250 5300 4150
-Wire Wire Line
-	5300 4150 6400 4150
 Wire Notes Line
 	7550 2850 7550 4650
@@
 Wire Wire Line
 	4500 5400 4500 5250
+$Comp
+L 8P8C_Shielded:8P8C_Shielded_Custom J1
+U 1 1 600A1FE7
+P 1900 2050
+F 0 "J1" H 1700 2600 50  0000 R CNN
+F 1 "Torch" H 1750 2700 50  0000 R CNN
+F 2 "RJHSE-3380:RJHSE3384" V 1900 2075 50  0001 C CNN
+F 3 "https://datasheet.lcsc.com/szlcsc/1811141123_Shanghai-YDS-Tech-51F-1210GY2D2NL_C179768.pdf" V 1900 2075 50  0001 C CNN
+F 4 "C179768" H 1900 2050 50  0001 C CNN "LCSC"
+F 5 "51F-1210GY2D2NL" H 1900 2050 50  0001 C CNN "PN"
+	1    1900 2050
+	1    0    0    -1
+$EndComp
+$Comp
+L 8P8C_Shielded:8P8C_Shielded_Custom J8
+U 1 1 6023A990
+P 5800 4250
+F 0 "J8" H 5600 4800 50  0000 R CNN
+F 1 "Torch" H 5650 4900 50  0000 R CNN
+F 2 "RJHSE-3380:RJHSE3384" V 5800 4275 50  0001 C CNN
+F 3 "https://datasheet.lcsc.com/szlcsc/1811141123_Shanghai-YDS-Tech-51F-1210GY2D2NL_C179768.pdf" V 5800 4275 50  0001 C CNN
+F 4 "C179768" H 5800 4250 50  0001 C CNN "LCSC"
+F 5 "51F-1210GY2D2NL" H 5800 4250 50  0001 C CNN "PN"
+	1    5800 4250
+	0    1    -1   0
+$EndComp
+$Comp
+L 8P8C_Shielded:8P8C_Shielded_Custom J4
+U 1 1 600B48EF
+P 8150 1550
+F 0 "J4" H 7950 2100 50  0000 R CNN
+F 1 "Limit" H 8000 2200 50  0000 R CNN
+F 2 "RJHSE-3380:RJHSE3384" V 8150 1575 50  0001 C CNN
+F 3 "https://datasheet.lcsc.com/szlcsc/1811141123_Shanghai-YDS-Tech-51F-1210GY2D2NL_C179768.pdf" V 8150 1575 50  0001 C CNN
+F 4 "C179768" H 8150 1550 50  0001 C CNN "LCSC"
+F 5 "51F-1210GY2D2NL" H 8150 1550 50  0001 C CNN "PN"
+	1    8150 1550
+	1    0    0    -1
+$EndComp
+Wire Wire Line
+	7600 1900 7650 1900
+Wire Wire Line
+	7600 1900 7600 1800
+Wire Wire Line
+	7600 1800 7650 1800
+Connection ~ 7600 1900
+Wire Wire Line
+	7600 1800 7600 1200
+Wire Wire Line
+	7600 1200 7650 1200
+Connection ~ 7600 1800
+Wire Wire Line
+	7600 1200 7600 1100
+Wire Wire Line
+	7600 1100 7650 1100
+Connection ~ 7600 1200
+Wire Wire Line
+	5450 4750 5450 4800
+Wire Wire Line
+	5450 4800 5550 4800
+Wire Wire Line
+	6250 4750 6250 4800
+Connection ~ 6250 4800
+Wire Wire Line
+	6150 4750 6150 4800
+Connection ~ 6150 4800
+Wire Wire Line
+	6150 4800 6250 4800
+Wire Wire Line
+	5550 4750 5550 4800
+Connection ~ 5550 4800
+Wire Wire Line
+	5550 4800 6150 4800
+Wire Wire Line
+	1400 1600 1350 1600
+Wire Wire Line
+	1350 1600 1350 1700
+Wire Wire Line
+	1350 1700 1400 1700
+Wire Wire Line
+	1350 1700 1350 2300
+Connection ~ 1350 1700
+Wire Wire Line
+	1400 2300 1350 2300
+Connection ~ 1350 2300
+Wire Wire Line
+	1350 2300 1350 2400
+Wire Wire Line
+	1400 2400 1350 2400
+Connection ~ 1350 2400
+Wire Wire Line
+	1900 2650 1350 2650
+Wire Wire Line
+	1350 2400 1350 2650
+Connection ~ 1900 2650
+Wire Wire Line
+	6400 4250 6400 4800
+Wire Wire Line
+	6250 4800 6400 4800
+Connection ~ 6400 4250
+Wire Wire Line
+	5300 4250 5250 4250
+Wire Wire Line
+	5250 4250 5250 4150
+Wire Wire Line
+	5250 4150 6400 4150
+Wire Wire Line
+	8150 2050 7600 2050
+Wire Wire Line
+	7600 1900 7600 2050
+Connection ~ 8150 2050
+$Comp
+L Mechanical:MountingHole H1
+U 1 1 60B08E8A
+P 7400 -1050
+F 0 "H1" H 7500 -1004 50  0000 L CNN
+F 1 "MountingHole" H 7500 -1095 50  0000 L CNN
+F 2 "MountingHole:MountingHole_3.2mm_M3" H 7400 -1050 50  0001 C CNN
+F 3 "~" H 7400 -1050 50  0001 C CNN
+	1    7400 -1050
+	1    0    0    -1
+$EndComp
+$Comp
+L Mechanical:MountingHole H2
+U 1 1 60B5F657
+P 7400 -800
+F 0 "H2" H 7500 -754 50  0000 L CNN
+F 1 "MountingHole" H 7500 -845 50  0000 L CNN
+F 2 "MountingHole:MountingHole_3.2mm_M3" H 7400 -800 50  0001 C CNN
+F 3 "~" H 7400 -800 50  0001 C CNN
+	1    7400 -800
+	1    0    0    -1
+$EndComp
 $EndSCHEMATC

Commit message: Added RJ45 Clearpath BOB, minor torch module footprint fix
Parts:
- removed Q2, Q3, Q4, Q5: IRLML2402, Package_TO_SOT_SMD:SOT-23, symbol Device:Q_NMOS_GDS
- added Q2, Q3, Q4, Q5: IRLML2402, Package_TO_SOT_SMD:SOT-23, symbol Device:Q_NMOS_GSD
- J1, J4, J8: symbol 8P8C_Shielded:8P8C_Shielded_Custom -> Torch-Module-rescue:8P8C_Shielded_Custom-8P8C_Shielded
- J6: symbol Torch_Module-cache:My_library_8P8C_LED_Shielded -> Torch-Module-rescue:My_library_8P8C_LED_Shielded-Torch_Module-cache
Connections:
- net at J11.11 (Pin_11): now also Q5.3 (D)
- net at J11.12 (Pin_12): now also Q3.3 (D)
- net at J11.13 (Pin_13): now also Q4.3 (D)
- net at J11.14 (Pin_14): now also Q2.3 (D)
- net at J11.15 (Pin_15), J11.9 (Pin_9), R17.2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: now also Q2.2 (S), Q3.2 (S), Q4.2 (S), Q5.2 (S)
- net at R8.2, R9.1: now also Q2.1 (G)
- net at R18.2, R19.1: now also Q4.1 (G)
- net at R10.2, R17.1: now also Q3.1 (G)
- net at R20.2, R21.1: now also Q5.1 (G)
Changed lines of the file:
@@
-$EndComp
-$Comp
-L Device:Q_NMOS_GDS Q2
-U 1 1 601F7D6C
-P 8400 5150
-F 0 "Q2" H 8604 5196 50  0000 L CNN
-F 1 "IRLML2402" H 8604 5105 50  0000 L CNN
-F 2 "Package_TO_SOT_SMD:SOT-23" H 8600 5250 50  0001 C CNN
-F 3 "~" H 8400 5150 50  0001 C CNN
-F 4 "C2588" H 8400 5150 50  0001 C CNN "LCSC"
-F 5 "IRLML2402TRPBF" H 8400 5150 50  0001 C CNN "PN"
-	1    8400 5150
-	1    0    0    -1
 $EndComp
 $Comp
@@
 Connection ~ 8200 5150
 $Comp
-L Device:Q_NMOS_GDS Q4
-U 1 1 6020F226
-P 9700 5150
-F 0 "Q4" H 9904 5196 50  0000 L CNN
-F 1 "IRLML2402" H 9904 5105 50  0000 L CNN
-F 2 "Package_TO_SOT_SMD:SOT-23" H 9900 5250 50  0001 C CNN
-F 3 "~" H 9700 5150 50  0001 C CNN
-F 4 "C2588" H 9700 5150 50  0001 C CNN "LCSC"
-F 5 "IRLML2402TRPBF" H 9700 5150 50  0001 C CNN "PN"
-	1    9700 5150
-	1    0    0    -1
-$EndComp
-$Comp
 L Device:R_US R19
 U 1 1 6020F908
@@
 	1    0    0    -1
 $EndComp
-Connection ~ 9500 5150
-$Comp
-L Device:Q_NMOS_GDS Q3
-U 1 1 6022166D
-P 8400 5900
-F 0 "Q3" H 8604 5946 50  0000 L CNN
-F 1 "IRLML2402" H 8604 5855 50  0000 L CNN
-F 2 "Package_TO_SOT_SMD:SOT-23" H 8600 6000 50  0001 C CNN
-F 3 "~" H 8400 5900 50  0001 C CNN
-F 4 "C2588" H 8400 5900 50  0001 C CNN "LCSC"
-F 5 "IRLML2402TRPBF" H 8400 5900 50  0001 C CNN "PN"
-	1    8400 5900
-	1    0    0    -1
-$EndComp
 $Comp
 L Device:R_US R17
@@
 	1    0    0    -1
 $EndComp
-Connection ~ 8200 5900
-$Comp
-L Device:Q_NMOS_GDS Q5
-U 1 1 6022FF01
-P 9700 5900
-F 0 "Q5" H 9904 5946 50  0000 L CNN
-F 1 "IRLML2402" H 9904 5855 50  0000 L CNN
-F 2 "Package_TO_SOT_SMD:SOT-23" H 9900 6000 50  0001 C CNN
-F 3 "~" H 9700 5900 50  0001 C CNN
-F 4 "C2588" H 9700 5900 50  0001 C CNN "LCSC"
-F 5 "IRLML2402TRPBF" H 9700 5900 50  0001 C CNN "PN"
-	1    9700 5900
-	1    0    0    -1
-$EndComp
 $Comp
 L Device:R_US R21
@@
 	1    0    0    -1
 $EndComp
-Connection ~ 9500 5900
 Wire Wire Line
 	8050 4550 8050 4850
@@
 	8550 2900 8900 2900
 $Comp
-L Torch_Module-cache:My_library_8P8C_LED_Shielded J6
+L Torch-Module-rescue:My_library_8P8C_LED_Shielded-Torch_Module-cache J6
 U 1 1 6026066F
 P 9400 3200
@@
 	4500 5400 4500 5250
 $Comp
-L 8P8C_Shielded:8P8C_Shielded_Custom J1
+L Torch-Module-rescue:8P8C_Shielded_Custom-8P8C_Shielded J1
 U 1 1 600A1FE7
 P 1900 2050
@@
 $EndComp
 $Comp
-L 8P8C_Shielded:8P8C_Shielded_Custom J8
+L Torch-Module-rescue:8P8C_Shielded_Custom-8P8C_Shielded J8
 U 1 1 6023A990
 P 5800 4250
@@
 $EndComp
 $Comp
-L 8P8C_Shielded:8P8C_Shielded_Custom J4
+L Torch-Module-rescue:8P8C_Shielded_Custom-8P8C_Shielded J4
 U 1 1 600B48EF
 P 8150 1550
@@
 	1    0    0    -1
 $EndComp
+Connection ~ 9500 5150
+$Comp
+L Device:Q_NMOS_GSD Q2
+U 1 1 618B4EB4
+P 8400 5150
+F 0 "Q2" H 8604 5196 50  0000 L CNN
+F 1 "IRLML2402" H 8604 5105 50  0000 L CNN
+F 2 "Package_TO_SOT_SMD:SOT-23" H 8600 5250 50  0001 C CNN
+F 3 "~" H 8400 5150 50  0001 C CNN
+F 4 "C2588" H 8400 5150 50  0001 C CNN "LCSC"
+F 5 "IRLML2402TRPBF" H 8400 5150 50  0001 C CNN "PN"
+	1    8400 5150
+	1    0    0    -1
+$EndComp
+$Comp
+L Device:Q_NMOS_GSD Q4
+U 1 1 618B65D2
+P 9700 5150
+F 0 "Q4" H 9904 5196 50  0000 L CNN
+F 1 "IRLML2402" H 9904 5105 50  0000 L CNN
+F 2 "Package_TO_SOT_SMD:SOT-23" H 9900 5250 50  0001 C CNN
+F 3 "~" H 9700 5150 50  0001 C CNN
+F 4 "C2588" H 9700 5150 50  0001 C CNN "LCSC"
+F 5 "IRLML2402TRPBF" H 9700 5150 50  0001 C CNN "PN"
+	1    9700 5150
+	1    0    0    -1
+$EndComp
+$Comp
+L Device:Q_NMOS_GSD Q5
+U 1 1 618B755A
+P 9700 5900
+F 0 "Q5" H 9904 5946 50  0000 L CNN
+F 1 "IRLML2402" H 9904 5855 50  0000 L CNN
+F 2 "Package_TO_SOT_SMD:SOT-23" H 9900 6000 50  0001 C CNN
+F 3 "~" H 9700 5900 50  0001 C CNN
+F 4 "C2588" H 9700 5900 50  0001 C CNN "LCSC"
+F 5 "IRLML2402TRPBF" H 9700 5900 50  0001 C CNN "PN"
+	1    9700 5900
+	1    0    0    -1
+$EndComp
+Connection ~ 9500 5900
+$Comp
+L Device:Q_NMOS_GSD Q3
+U 1 1 618B85D4
+P 8400 5900
+F 0 "Q3" H 8604 5946 50  0000 L CNN
+F 1 "IRLML2402" H 8604 5855 50  0000 L CNN
+F 2 "Package_TO_SOT_SMD:SOT-23" H 8600 6000 50  0001 C CNN
+F 3 "~" H 8400 5900 50  0001 C CNN
+F 4 "C2588" H 8400 5900 50  0001 C CNN "LCSC"
+F 5 "IRLML2402TRPBF" H 8400 5900 50  0001 C CNN "PN"
+	1    8400 5900
+	1    0    0    -1
+$EndComp
+Connection ~ 8200 5900
 $EndSCHEMATC
