File: Hardware/Torch Module/Torch Module.kicad_sch (KiCad schematic)
At the start: 84 parts, among them J1 Torch, J4 Limit, J6 8P8C_LED_Shielded, J8 Torch

Commit message: Pin Naming Changes
Parts:
- gave numbers to parts that had none: 78
Connections:
- net at J14.2 (Pin_2), J2.10 (Pin_10): now also J2.5 (Pin_5)
- no-connect marks 42 -> 41
Other:
- note added: "Report"
- note added: "Torch IO 36 THC Report"
- note removed: "Torch IO 36 THC"
