File: Hardware/Clearpath MotorDriver Mosfet/Clearpath MotorDriver Mosfet.kicad_pcb (KiCad board)
At the start: 2 copper layers, 16.1 x 20.4 mm, 13 parts, among them J1 Conn_01x18_Male, Q1 IRLML2402, Q2 IRLML2402, Q3 IRLML2402, Q4 IRLML2402

Commit message: Gerber Upload Ordered version
Changed lines of the file:
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@@
       (layerselection 0x00010fc_ffffffff)
       (disableapertmacros false)
-      (usegerberextensions false)
-      (usegerberattributes true)
-      (usegerberadvancedattributes true)
-      (creategerberjobfile true)
+      (usegerberextensions true)
+      (usegerberattributes false)
+      (usegerberadvancedattributes false)
+      (creategerberjobfile false)
       (svguseinch false)
       (svgprecision 6)
@@
       (psa4output false)
       (plotreference true)
-      (plotvalue true)
+      (plotvalue false)
       (plotinvisibletext false)
       (sketchpadsonfab false)
-      (subtractmaskfromsilk false)
+      (subtractmaskfromsilk true)
       (outputformat 1)
       (mirror false)
-      (drillshape 1)
+      (drillshape 0)
       (scaleselection 1)
-      (outputdirectory "")
+      (outputdirectory "gerber/")
     )
   )
@@
     (property "Sheetname" "")
     (attr smd)
-    (fp_text reference "Q2" (at 0 -2.4) (layer "F.SilkS")
+    (fp_text reference "Q2" (at 1.405 -1.482 90) (layer "F.SilkS")
       (effects (font (size 1 1) (thickness 0.15)))
     )
@@
     (property "Sheetname" "")
     (attr smd)
-    (fp_text reference "R1" (at 0 -1.43 90) (layer "F.SilkS")
-      (effects (font (size 1 1) (thickness 0.15)))
+    (fp_text reference "R1" (at 0.104 -0.062 -270) (layer "B.SilkS")
+      (effects (font (size 1 1) (thickness 0.15)) (justify mirror))
     )
     (fp_text value "200" (at 0 1.43 90) (layer "F.Fab")
@@
     (property "Sheetname" "")
     (attr smd)
-    (fp_text reference "R5" (at 0 -1.43 90) (layer "F.SilkS")
-      (effects (font (size 1 1) (thickness 0.15)))
+    (fp_text reference "R5" (at 0.142 -0.032 -270) (layer "B.SilkS")
+      (effects (font (size 1 1) (thickness 0.15)) (justify mirror))
     )
     (fp_text value "200" (at 0 1.43 90) (layer "F.Fab")
@@
     (property "Sheetname" "")
     (attr smd)
-    (fp_text reference "Q4" (at 0 -2.4) (layer "F.SilkS")
-      (effects (font (size 1 1) (thickness 0.15)))
-    )
-    (fp_text value "IRLML2402" (at 0 2.4) (layer "F.Fab")
+    (fp_text reference "Q4" (at 1.385 -1.643 90) (layer "F.SilkS")
+      (effects (font (size 1 1) (thickness 0.15)))
+    )
+    (fp_text value "IRLML2402" (at -2.615 2.567) (layer "F.Fab")
       (effects (font (size 1 1) (thickness 0.15)))
     )
@@
     (property "Sheetname" "")
     (attr smd)
-    (fp_text reference "Q1" (at 0 -2.4) (layer "F.SilkS")
+    (fp_text reference "Q1" (at 1.395 -1.494 90) (layer "F.SilkS")
       (effects (font (size 1 1) (thickness 0.15)))
     )
@@
     (property "Sheetname" "")
     (attr smd)
-    (fp_text reference "R6" (at 0 -1.43 90) (layer "F.SilkS")
-      (effects (font (size 1 1) (thickness 0.15)))
+    (fp_text reference "R6" (at -0.055 0.009 90) (layer "B.SilkS")
+      (effects (font (size 1 1) (thickness 0.15)) (justify mirror))
     )
     (fp_text value "10K" (at 0 -1.143 90) (layer "F.Fab")
@@
     (property "Sheetname" "")
     (attr smd)
-    (fp_text reference "R2" (at 0 -1.43 90) (layer "F.SilkS")
-      (effects (font (size 1 1) (thickness 0.15)))
+    (fp_text reference "R2" (at 0.096 -0.011 90) (layer "B.SilkS")
+      (effects (font (size 1 1) (thickness 0.15)) (justify mirror))
     )
     (fp_text value "10K" (at 0.127 -1.143 90) (layer "F.Fab")
@@
     (property "Sheetname" "")
     (attr smd)
-    (fp_text reference "Q3" (at 0 -2.4) (layer "F.SilkS")
+    (fp_text reference "Q3" (at 1.405 -1.545 90) (layer "F.SilkS")
       (effects (font (size 1 1) (thickness 0.15)))
     )
@@
     (property "Sheetname" "")
     (attr smd)
-    (fp_text reference "R4" (at 0 -1.43 90) (layer "F.SilkS")
-      (effects (font (size 1 1) (thickness 0.15)))
+    (fp_text reference "R4" (at 0.028 0.099 90) (layer "B.SilkS")
+      (effects (font (size 1 1) (thickness 0.15)) (justify mirror))
     )
     (fp_text value "10K" (at 0.127 -1.143 90) (layer "F.Fab")
@@
     (property "Sheetname" "")
     (attr through_hole)
-    (fp_text reference "J1" (at -0.762 10.414 180) (layer "F.SilkS")
+    (fp_text reference "J1" (at -0.953 9.024 180) (layer "F.SilkS")
       (effects (font (size 1 1) (thickness 0.15)))
     )
@@
     (property "Sheetname" "")
     (attr smd)
-    (fp_text reference "R7" (at 0 -1.43 90) (layer "F.SilkS")
+    (fp_text reference "R7" (at -2.557 -0.082 90) (layer "F.SilkS")
       (effects (font (size 1 1) (thickness 0.15)))
     )
@@
     (property "Sheetname" "")
     (attr smd)
-    (fp_text reference "R3" (at 0 -1.43 90) (layer "F.SilkS")
-      (effects (font (size 1 1) (thickness 0.15)))
+    (fp_text reference "R3" (at -0.081 -0.022 -270) (layer "B.SilkS")
+      (effects (font (size 1 1) (thickness 0.15)) (justify mirror))
     )
     (fp_text value "200" (at 0 1.43 90) (layer "F.Fab")
@@
     (property "Sheetname" "")
     (attr smd)
-    (fp_text reference "R8" (at 0 -1.43 90) (layer "F.SilkS")
+    (fp_text reference "R8" (at 2.537 0.099 90) (layer "F.SilkS")
       (effects (font (size 1 1) (thickness 0.15)))
     )
@@
   (segment (start 93.98 92.71) (end 93.98 91.694) (width 1) (layer "F.Cu") (net 11))
   (segment (start 93.98 91.694) (end 94.107 91.567) (width 1) (layer "F.Cu") (net 11))
-  (segment (start 102.0845 98.679) (end 102.108 98.6555) (width 0.25) (layer "F.Cu") (net 14))
-  (segment (start 101.473 98.679) (end 102.0845 98.679) (width 0.25) (layer "F.Cu") (net 14))
-  (segment (start 100.965 98.171) (end 101.473 98.679) (width 0.25) (layer "F.Cu") (net 14))
-  (segment (start 100.965 97.917) (end 100.965 98.171) (width 0.25) (layer "F.Cu") (net 14))
-  (via (at 100.965 97.917) (size 0.8) (drill 0.4) (layers "F.Cu" "B.Cu") (net 14))
-  (segment (start 100.838 97.917) (end 100.965 97.917) (width 0.25) (layer "B.Cu") (net 14))
+  (segment (start 101.1425 97.69) (end 102.108 98.6555) (width 0.25) (layer "F.Cu") (net 14))
+  (segment (start 100.95 97.69) (end 101.1425 97.69) (width 0.25) (layer "F.Cu") (net 14))
+  (via (at 100.95 97.69) (size 0.8) (drill 0.4) (layers "F.Cu" "B.Cu") (net 14))
+  (segment (start 101.981 92.583) (end 101.981 96.669) (width 0.25) (layer "B.Cu") (net 14))
+  (segment (start 101.981 96.669) (end 100.95 97.7) (width 0.25) (layer "B.Cu") (net 14))
   (segment (start 103.078 91.486) (end 101.981 92.583) (width 0.25) (layer "B.Cu") (net 14))
-  (segment (start 101.6 97.282) (end 100.965 97.917) (width 0.25) (layer "B.Cu") (net 14))
-  (segment (start 101.981 96.901) (end 101.6 97.282) (width 0.25) (layer "B.Cu") (net 14))
-  (segment (start 101.981 92.583) (end 101.981 96.901) (width 0.25) (layer "B.Cu") (net 14))
+  (segment (start 100.95 97.7) (end 100.95 97.69) (width 0.25) (layer "B.Cu") (net 14))
   (segment (start 104.723 91.486) (end 103.078 91.486) (width 0.25) (layer "B.Cu") (net 14))
   (segment (start 102.0045 94.615) (end 102.108 94.7185) (width 0.25) (layer "F.Cu") (net 15))
