File: Hardware/Clearpath MotorDriver Mosfet/Clearpath MotorDriver Mosfet.kicad_sch (KiCad schematic)
At the start: 13 parts, among them J1 Conn_01x18_Male, Q1 IRLML2402, Q2 IRLML2402, Q3 IRLML2402, Q4 IRLML2402

Commit message: Updates from Nov 11
Parts:
- Q1, Q2, Q3, Q4: value IRLML2402 -> BSS138
Changed lines of the file:
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@@
       (effects (font (size 1.27 1.27)) (justify left))
     )
-    (property "Value" "IRLML2402" (id 1) (at 127.1016 86.233 0)
+    (property "Value" "BSS138" (id 1) (at 127.1016 86.233 0)
       (effects (font (size 1.27 1.27)) (justify left))
     )
@@
       (effects (font (size 1.27 1.27)) (justify left))
     )
-    (property "Value" "IRLML2402" (id 1) (at 160.1216 105.283 0)
+    (property "Value" "BSS138" (id 1) (at 160.1216 105.283 0)
       (effects (font (size 1.27 1.27)) (justify left))
     )
@@
       (effects (font (size 1.27 1.27)) (justify left))
     )
-    (property "Value" "IRLML2402" (id 1) (at 160.1216 86.233 0)
+    (property "Value" "BSS138" (id 1) (at 160.1216 86.233 0)
       (effects (font (size 1.27 1.27)) (justify left))
     )
@@
       (effects (font (size 1.27 1.27)) (justify left))
     )
-    (property "Value" "IRLML2402" (id 1) (at 127.1016 105.283 0)
+    (property "Value" "BSS138" (id 1) (at 127.1016 105.283 0)
       (effects (font (size 1.27 1.27)) (justify left))
     )
@@
     )
     (path "/32d9a73d-1c66-4298-878f-714343fd0cae"
-      (reference "Q1") (unit 1) (value "IRLML2402") (footprint "Package_TO_SOT_SMD:SOT-23")
+      (reference "Q1") (unit 1) (value "BSS138") (footprint "Package_TO_SOT_SMD:SOT-23")
     )
     (path "/990f80ca-21fe-4b7e-836a-c294e897c9a8"
-      (reference "Q2") (unit 1) (value "IRLML2402") (footprint "Package_TO_SOT_SMD:SOT-23")
+      (reference "Q2") (unit 1) (value "BSS138") (footprint "Package_TO_SOT_SMD:SOT-23")
     )
     (path "/8e849722-ebec-4d01-8989-1e6b1ba1caa4"
-      (reference "Q3") (unit 1) (value "IRLML2402") (footprint "Package_TO_SOT_SMD:SOT-23")
+      (reference "Q3") (unit 1) (value "BSS138") (footprint "Package_TO_SOT_SMD:SOT-23")
     )
     (path "/40ee0d66-7b3b-473d-9067-5cf5aba724a6"
-      (reference "Q4") (unit 1) (value "IRLML2402") (footprint "Package_TO_SOT_SMD:SOT-23")
+      (reference "Q4") (unit 1) (value "BSS138") (footprint "Package_TO_SOT_SMD:SOT-23")
     )
     (path "/f0aadf09-b0c1-48d7-80f4-5996f1cb1b10"
