File: Hardware/Main Board V2.0/Main Board/Main Board.kicad_sch (KiCad schematic)
At the start: 125 parts, among them J10 Conn_01x04, J11 Conn_01x04, J12 Conn_01x04, J16 Micro_SD_Card, J6 Module A1, J6 Module A2, J6 Module A3, J6 Module B1, J6 Module B2, J6 Module B3, J7 Conn_01x04, J8 Conn_01x04, J9 Conn_01x04, Q3 MMBT2222, Q4 MMBT2222, Q5 MMBT2222, Q6 MMBT2222, SW1 SW_Push, SW2 SW_Push, U10 GT-USB-7051A, U11 AP2112K-3.3, U12 AP2112K-3.3, U5 74AHCT595, U5 ESP32-WROOM-32UE-H4, U6 74AHCT595, U6 ESP32-WROOM-32UE-H4, U7 74AHCT595, U7 CP2104, U8 74AHCT595, U8 CP2104, U9 GT-USB-7051A

Commit message: Level shifters for motors roughed in, discover V1.1 issues with overcurrent on outputs
Parts:
- removed U5, U6, U7, U8: 74AHCT595, Package_SO:SO-16_5.3x10.2mm_P1.27mm, symbol 74xx:74AHCT595
- added Q1 (x18): BSS138, Package_TO_SOT_SMD:SOT-23, symbol Device:Q_NMOS_GSD
- added R35, R40, R43, R50, R51, R52, R59, R60, R61, R68, R69, R70, R77, R78, R79, R86, R87, R88: 200R, Resistor_SMD:R_0603_1608Metric, symbol Device:R_Small
- added R36, R39, R42, R47, R48, R49, R56, R57, R58, R65, R66, R67, R74, R75, R76, R83, R84, R85: 10K, Resistor_SMD:R_0603_1608Metric, symbol Device:R_Small
- added R37, R38, R41, R44, R45, R46, R53, R54, R55, R62, R63, R64, R71, R72, R73, R80, R81, R82: 500R, Resistor_SMD:R_0603_1608Metric, symbol Device:R_Small
- added U13, U14, U15, U16: 74AHCT595PW, Package_SO:TSSOP-16-1EP_4.4x5mm_P0.65mm, symbol 111_Torban_Symbols:74AHC595
Connections:
- net +5V: now also U13.10 (MR#), U13.16 (VCC), U14.10 (MR#), U14.16 (VCC), U15.10 (MR#), U15.16 (VCC), U16.10 (MR#), U16.16 (VCC)
- net A_Dir: now also R52.2, U14.4 (Q4)
- net A_Enable: now also R50.2, U14.7 (Q7)
- net A_Step: now also R51.2, U14.5 (Q5)
- net B_Dir: now also R61.2, U15.1 (Q1)
- net B_Enable: now also R59.2, U15.15 (Q0)
- net B_Step: now also R60.2, U15.2 (Q2)
- net C_Dir: now also R88.2, U15.4 (Q4)
- net C_Enable: now also R86.2, U15.7 (Q7)
- net C_Step: now also R87.2, U15.5 (Q5)
- net GND: now also Q1.2 (S), Q1.2 (S), Q1.2 (S), Q1.2 (S), Q1.2 (S), Q1.2 (S), Q1.2 (S), Q1.2 (S), Q1.2 (S), Q1.2 (S), Q1.2 (S), Q1.2 (S), Q1.2 (S), Q1.2 (S), Q1.2 (S), Q1.2 (S), Q1.2 (S), Q1.2 (S), R36.1, R39.1, R42.1, R47.1, R48.1, R49.1, R56.1, R57.1, R58.1, R65.1, R66.1, R67.1, R74.1, R75.1, R76.1, R83.1, R84.1, R85.1, U13.13 (OE#), U13.8 (GND), U14.13 (OE#), U14.8 (GND), U15.13 (OE#), U15.8 (GND), U16.13 (OE#), U16.8 (GND)
- net X_Dir: now also R43.2, U13.1 (Q1)
- net X_Enable: now also R35.2, U13.15 (Q0)
- net X_Step: now also R40.2, U13.2 (Q2)
- net Y_Dir: now also R70.2, U13.4 (Q4)
- net Y_Enable: now also R68.2, U13.7 (Q7)
- net Y_Step: now also R69.2, U13.5 (Q5)
- net Z_Dir: now also R79.2, U14.1 (Q1)
- net Z_Enable: now also R77.2, U14.15 (Q0)
- net Z_Steo renamed Z_Step
- net Z_Step: now also R78.2, U14.2 (Q2)
- new net: Q1.1 (G), R39.2, R40.1
- new net: Q1.1 (G), R35.1, R36.2
- new net: Q1.3 (D), R37.2
- new net: Q1.3 (D), R80.2
- new net: Q1.1 (G), R42.2, R43.1
- new net: Q1.1 (G), R75.2, R78.1
- new net: Q1.1 (G), R76.2, R79.1
- new net: Q1.3 (D), R73.2
- new net: U13.9 (Q7S), U14.14 (DS)
- new net: U14.9 (Q7S), U15.14 (DS)
- new net: Q1.1 (G), R57.2, R60.1
- new net: Q1.3 (D), R54.2
- new net: Q1.3 (D), R44.2
- new net: Q1.1 (G), R84.2, R87.1
- new net: Q1.1 (G), R66.2, R69.1
- new net: Q1.3 (D), R63.2
- new net: Q1.3 (D), R38.2
- new net: Q1.3 (D), R64.2
- new net: U15.9 (Q7S), U16.14 (DS)
- new net: Q1.1 (G), R48.2, R51.1
- new net: Q1.1 (G), R74.2, R77.1
- new net: Q1.3 (D), R62.2
- new net: Q1.1 (G), R67.2, R70.1
- new net: Q1.1 (G), R47.2, R50.1
- new net: Q1.3 (D), R82.2
- new net: Q1.1 (G), R83.2, R86.1
- new net: Q1.3 (D), R71.2
- new net: Q1.3 (D), R41.2
- new net: Q1.1 (G), R56.2, R59.1
- new net: Q1.1 (G), R65.2, R68.1
- new net: Q1.1 (G), R58.2, R61.1
- new net: Q1.3 (D), R55.2
- new net: Q1.3 (D), R72.2
- new net: Q1.3 (D), R46.2
- new net: Q1.1 (G), R85.2, R88.1
- new net: Q1.1 (G), R49.2, R52.1
- new net: Q1.3 (D), R53.2
- new net: Q1.3 (D), R45.2
- new net: Q1.3 (D), R81.2
- new net A_Dir_HV: R46.1
- new net A_Enable_HV: R44.1
- new net A_Step_HV: R45.1
- new net B_Dir_HV: R55.1
- new net B_Enable_HV: R53.1
- new net B_Step_HV: R54.1
- new net C_Dir_HV: R82.1
- new net C_Enable_HV: R80.1
- new net C_Step_HV: R81.1
- new net I2S0_11: U14.3 (Q3)
- new net I2S0_14: U14.6 (Q6)
- new net I2S0_19: U15.3 (Q3)
- new net I2S0_22: U15.6 (Q6)
- new net I2S0_24: U16.15 (Q0)
- new net I2S0_25: U16.1 (Q1)
- new net I2S0_26: U16.2 (Q2)
- new net I2S0_27: U16.3 (Q3)
- new net I2S0_28: U16.4 (Q4)
- new net I2S0_29: U16.5 (Q5)
- new net I2S0_3: U13.3 (Q3)
- new net I2S0_30: U16.6 (Q6)
- new net I2S0_31: U16.7 (Q7)
- new net I2S0_6: U13.6 (Q6)
- new net I2S_BCK: U13.11 (SHCP), U14.11 (SHCP), U15.11 (SHCP), U16.11 (SHCP)
- new net I2S_DATA: U13.14 (DS)
- new net I2S_WS: U13.12 (STCP), U14.12 (STCP), U15.12 (STCP), U16.12 (STCP)
- new net X_Dir_HV: R41.1
- new net X_Enable_HV: R37.1
- new net X_Step_HV: R38.1
- new net Y_Dir_HV: R64.1
- new net Y_Enable_HV: R62.1
- new net Y_Step_HV: R63.1
- new net Z_Dir_HV: R73.1
- new net Z_Enable_HV: R71.1
- new net Z_Step_HV: R72.1
- no-connect marks 28 -> 29
Other:
- moved on the sheet: D1, D10, D11, D12, D13, D14, D15, D16, D17, D18, D2, D3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

Commit message: Organize, add mux, mapping and figuring out modules
Parts:
- removed D10, D11, D12, D13, D14, D15, D16, D17, D18, D2, D3, D4, D5, D6, D7, D8, D9: LED_Small_Filled, symbol Device:LED_Small_Filled
- removed J10, J11, J12, J7, J8, J9: Conn_01x04, symbol Connector_Generic:Conn_01x04
- removed J6: Module A2, Connector_PinSocket_2.54mm:PinSocket_1x12_P2.54mm_Vertical, symbol BDringController-rescue:IO_connector-My_Library-BDringController-rescue
- removed J6: Module A3, Connector_PinSocket_2.54mm:PinSocket_1x12_P2.54mm_Vertical, symbol BDringController-rescue:IO_connector-My_Library-BDringController-rescue
- removed J6: Module B3, Connector_PinSocket_2.54mm:PinSocket_1x12_P2.54mm_Vertical, symbol BDringController-rescue:IO_connector-My_Library-BDringController-rescue
- removed J6: Module B2, Connector_PinSocket_2.54mm:PinSocket_1x12_P2.54mm_Vertical, symbol BDringController-rescue:IO_connector-My_Library-BDringController-rescue
- removed J6: Module A1, Connector_PinSocket_2.54mm:PinSocket_1x12_P2.54mm_Vertical, symbol BDringController-rescue:IO_connector-My_Library-BDringController-rescue
- removed J6: Module B1, Connector_PinSocket_2.54mm:PinSocket_1x12_P2.54mm_Vertical, symbol BDringController-rescue:IO_connector-My_Library-BDringController-rescue
- removed R21, R22: 4.3K, Resistor_SMD:R_0603_1608Metric, symbol Device:R_Small
- added C26: 100nF, Capacitor_SMD:C_0603_1608Metric, symbol Device:C_Small
- added D23, D24, D27, D28, D29, D30, D31, D32, D33, D34, D35, D36, D37, D38, D39, D40, D41: LED_Small_Filled, symbol Device:LED_Small_Filled
- added J2 (x6): Screw_Terminal_01x06, User Library:2x3 screw terminal3.5mm, symbol Connector:Screw_Terminal_01x06
- added R89, R90: 1K, Resistor_SMD:R_0603_1608Metric, symbol Device:R_Small
- added U1: 74LVC157A, Package_SO:SOP-16_3.9x9.9mm_P1.27mm, symbol 111_Torban_Symbols:74LVC157A
- added U17: Module A3, Connector_PinSocket_2.54mm:PinSocket_1x12_P2.54mm_Vertical, symbol 111_Torban_Symbols:BDring_IO_Module
- added U18: Module B1, Connector_PinSocket_2.54mm:PinSocket_1x12_P2.54mm_Vertical, symbol 111_Torban_Symbols:BDring_IO_Module
- added U19: Module B2, Connector_PinSocket_2.54mm:PinSocket_1x12_P2.54mm_Vertical, symbol 111_Torban_Symbols:BDring_IO_Module
- added U20: Module B3, Connector_PinSocket_2.54mm:PinSocket_1x12_P2.54mm_Vertical, symbol 111_Torban_Symbols:BDring_IO_Module
- added U3: Module A1, Connector_PinSocket_2.54mm:PinSocket_1x12_P2.54mm_Vertical, symbol 111_Torban_Symbols:BDring_IO_Module
- added U4: Module A2, Connector_PinSocket_2.54mm:PinSocket_1x12_P2.54mm_Vertical, symbol 111_Torban_Symbols:BDring_IO_Module
- R10, R11, R12, R13, R14, R15, R16, R17, R18, R19, R20, R3, R4, R8, R9: value 4.3K -> 500R
- R38, R41, R46, R53, R54, R55, R62, R63, R64, R71, R72, R73, R80, R81, R82: value 500R -> 1K
- R7: value 4.3K -> 1K
Connections:
- net A_Dir_HV: now also Q1.3 (D), D29.1 (K), J2.3 (Pin_3); no longer R46.1
- net A_Enable: no longer R14.2
- net A_Enable_HV: now also Q1.3 (D), D27.1 (K), J2.1 (Pin_1); no longer R44.1
- net A_GPIO_17: no longer U6.28 (GPIO17)
- net A_MISO: now also U17.11 (8), U3.11 (8), U4.11 (8)
- net A_MOSI: now also U17.9 (6), U3.9 (6), U4.9 (6)
- net A_SCL: no longer U6.36 (GPIO22)
- net A_SCLK: now also U17.8 (5), U3.8 (5), U4.8 (5)
- net A_SDA: no longer U6.33 (GPIO21)
- net A_Step: no longer R15.2, R16.2
- net A_Step_HV: now also Q1.3 (D), D24.1 (K), J2.2 (Pin_2); no longer R45.1
- net A_VCC: now also U17.3 (VCC), U3.3 (VCC), U4.3 (VCC)
- net B_Dir_HV: now also Q1.3 (D), D35.1 (K), J2.3 (Pin_3); no longer R55.1
- net B_Enable: no longer R17.2
- net B_Enable_HV: now also Q1.3 (D), D31.1 (K), J2.1 (Pin_1); no longer R53.1
- net B_GPIO_18: no longer U5.30 (GPIO18)
- net B_GPIO_19: no longer U5.31 (GPIO19)
- net B_GPIO_23: no longer U5.37 (GPIO23)
- net B_GPIO_4: no longer U5.26 (ADC2_CH0/GPIO4)
- net B_MISO: now also U18.11 (8), U19.11 (8), U20.11 (8)
- net B_MOSI: now also U18.9 (6), U19.9 (6), U20.9 (6)
- net B_SCLK: now also U18.8 (5), U19.8 (5), U20.8 (5)
- net B_Step: no longer R18.2, R19.2
- net B_Step_HV: now also Q1.3 (D), D33.1 (K), J2.2 (Pin_2); no longer R54.1
- net B_VCC: now also C26.1, U1.16 (VCC), U18.3 (VCC), U19.3 (VCC)
- net C_Dir_HV: now also Q1.3 (D), D41.1 (K), J2.3 (Pin_3); no longer R82.1
- net C_Enable: no longer R20.2
- net C_Enable_HV: now also Q1.3 (D), D37.1 (K), J2.1 (Pin_1); no longer R80.1
- net C_Step_HV: now also Q1.3 (D), D39.1 (K), J2.2 (Pin_2); no longer R81.1
- net GND: now also C26.2, U1.15 (~{EN}), U1.8 (GND), U17.1 (Gnd), U17.12 (Gnd), U18.1 (Gnd), U18.12 (Gnd), U19.1 (Gnd), U19.12 (Gnd), U20.1 (Gnd), U20.12 (Gnd), U3.1 (Gnd), U3.12 (Gnd), U4.1 (Gnd), U4.12 (Gnd); no longer D1.1 (K)
- net I2S_BCK: now also U6.36 (GPIO22)
- net I2S_DATA: now also U6.33 (GPIO21)
- net I2S_WS: now also U6.28 (GPIO17)
- net Vdrive: now also R10.1, R11.1, R12.1, R13.1, R14.1, R15.1, R16.1, R17.1, R18.1, R19.1, R20.1, R3.1, R37.1, R38.2, R4.1, R41.2, R44.1, R45.1, R46.2, R53.2, R54.2, R55.2, R62.2, R63.2, R64.2, R7.2, R71.2, R72.2, R73.2, R8.1, R80.2, R81.2, R82.2, R9.1, R89.2, R90.2, U17.2 (VMot), U18.2 (VMot), U19.2 (VMot), U20.2 (VMot), U3.2 (VMot), U4.2 (VMot)
- net X_Dir_HV: now also Q1.3 (D), D28.1 (K), J2.3 (Pin_3); no longer R41.1
- net X_Enable: no longer R7.2
- net X_Enable_HV: now also D1.1 (K), Q1.3 (D), J2.1 (Pin_1); no longer R37.1
- net X_Step: no longer R3.2, R4.2
- net X_Step_HV: now also Q1.3 (D), D23.1 (K), J2.2 (Pin_2); no longer R38.1
- net Y_Dir_HV: now also Q1.3 (D), D34.1 (K), J2.3 (Pin_3); no longer R64.1
- net Y_Enable: no longer R8.2
- net Y_Enable_HV: now also Q1.3 (D), D30.1 (K), J2.1 (Pin_1); no longer R62.1
- net Y_Step: no longer R10.2, R9.2
- net Y_Step_HV: now also Q1.3 (D), D32.1 (K), J2.2 (Pin_2); no longer R63.1
- net Z_Dir: now also U1.7 (Qb); no longer U14.1 (Q1)
- net Z_Dir_HV: now also Q1.3 (D), D40.1 (K), J2.3 (Pin_3); no longer R73.1
- net Z_Enable: now also U1.4 (Qa); no longer R11.2, U14.15 (Q0)
- net Z_Enable_HV: now also Q1.3 (D), D36.1 (K), J2.1 (Pin_1); no longer R71.1
- net Z_Step: now also U1.9 (Qc); no longer R12.2, R13.2, U14.2 (Q2)
- net Z_Step_HV: now also Q1.3 (D), D38.1 (K), J2.2 (Pin_2); no longer R72.1
- net at R37.2: now also J2.5 (Pin_5); no longer Q1.3 (D)
- net at R44.2: now also J2.6 (Pin_6); no longer Q1.3 (D)
- net at R45.2: now also J2.4 (Pin_4); no longer Q1.3 (D)
- new net: J2.4 (Pin_4), R18.2
- new net: D31.2 (A), R62.1
- new net: D40.2 (A), R89.1
- new net: J2.5 (Pin_5), R16.2
- new net: J2.4 (Pin_4), R3.2
- new net: J2.5 (Pin_5), R4.2
- new net: J2.6 (Pin_6), R8.2
- new net: D23.2 (A), R38.1
- new net: D27.2 (A), R46.1
- new net: D37.2 (A), R80.1
- new net: J2.4 (Pin_4), R12.2
- new net: J2.4 (Pin_4), R9.2
- new net: J2.5 (Pin_5), R10.2
- new net: J2.6 (Pin_6), R11.2
- new net: J2.4 (Pin_4), R15.2
- new net: J2.6 (Pin_6), R17.2
- new net: J2.5 (Pin_5), R13.2
- new net: D32.2 (A), R63.1
- new net: D29.2 (A), R54.1
- new net: D36.2 (A), R73.1
- new net: J2.6 (Pin_6), R14.2
- new net: J2.5 (Pin_5), R19.2
- new net: D39.2 (A), R82.1
- new net: D24.2 (A), R41.1
- new net: J2.6 (Pin_6), R20.2
- new net: D33.2 (A), R64.1
- new net: D41.2 (A), R90.1
- new net: D35.2 (A), R72.1
- new net: D34.2 (A), R71.1
- new net: D30.2 (A), R55.1
- new net: D28.2 (A), R53.1
- new net: D38.2 (A), R81.1
- new net MUX_SET: U1.1 (S), U5.26 (ADC2_CH0/GPIO4)
- new net Z_Dir_GRBL: U1.5 (I0b), U14.1 (Q1)
- new net Z_Dir_THC: U1.6 (I1b), U5.30 (GPIO18)
- new net Z_Enable_GRBL: U1.2 (I0a), U14.15 (Q0)
- new net Z_Enable_THC: U1.3 (I1a), U5.31 (GPIO19)
- new net Z_Step_GRBL: U1.11 (I0c), U14.2 (Q2)
- new net Z_Step_THC: U1.10 (I1c), U5.37 (GPIO23)
- no-connect marks 29 -> 32
Other:
- note added: "12V SMPS Buck Supply (24V In)"
- note added: "Expansion Modules"
- note added: "FluidNC ESP32"
- note added: "Stepper Outputs & Level Shifting"
- note added: "Torch Control ESP32"
- moved on the sheet: C1, C10, C11, C12, C13, C14, C15, C16, C17, C18, C19, C2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

Commit message: Cleanup, add decoupling resistors
Parts:
- added C27, C28, C29, C30: 100nF, Capacitor_SMD:C_0603_1608Metric, symbol Device:C_Small
- added JP5, JP6: Jumper_3_Open, symbol Jumper:Jumper_3_Open
Connections:
- net +5V: now also C27.1, C28.1, C29.1, C30.1
- net A_SCL: now also JP6.1 (A)
- net A_SDA: now also JP5.1 (A)
- net GND: now also C27.2, C28.2, C29.2, C30.2
Other:
- note added: "3V3 ESP32 Voltage Regulators"
- note added: "5V SMPS Buck Supply"
- note added: "CoProcessor ESP32"
- note added: "Expansion Modules For CoProcessor"
- note added: "Expansion Modules For FluidNC"
- note removed: "Expansion Modules"
- note removed: "Torch Control ESP32"
- moved on the sheet: C14, C21, C22, C23, C24, C25, D1, D23, D24, D25, D26, D27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

Commit message: add comments for power supplies
Parts:
- removed JP5, JP6: Jumper_3_Open, symbol Jumper:Jumper_3_Open
- added J8: Conn_01x03, symbol Connector_Generic:Conn_01x03
- renumbered C12 to C1, C16 to C10, C21 to C11, C17 to C12, C22 to C13, C10 to C14, C23 to C15, C24 to C16, C25 to C17, C26 to C18, C13 to C19, C5 to C2, C7 to C20, C8 to C21, C18 to C22, C19 to C23, C20 to C24, C11 to C25, C4 to C26, C1 to C27, C9 to C28, C2 to C29, C6 to C3, C3 to C30, C27 to C4, C28 to C5, C29 to C6, C30 to C7, C14 to C8, C15 to C9, D27 to D10, D24 to D11, D29 to D12, D31 to D13, D33 to D14, D35 to D15, D37 to D16, D39 to D17, D41 to D18, D21 to D19, D23 to D2, D19 to D20, D25 to D21, D26 to D22, D22 to D23, D20 to D24, D28 to D3, D30 to D4, D32 to D5, D34 to D6, D36 to D7, D38 to D8, D40 to D9, JP3 to JP5, JP4 to JP6, Q5 to Q19, Q6 to Q20, Q3 to Q21, Q4 to Q22, R35 to R1, R7 to R10, R38 to R11, R53 to R12, R55 to R13, R63 to R14, R71 to R15, R73 to R16, R81 to R17, R89 to R18, R36 to R19, R40 to R2, R39 to R20, R42 to R21, R65 to R22, R66 to R23, R67 to R24, R74 to R25, R75 to R26, R76 to R27, R29 to R28, R50 to R29, R43 to R3, R51 to R30, R52 to R31, R59 to R32, R60 to R33, R61 to R34, R86 to R35, R87 to R36, R88 to R37, R46 to R38, R41 to R39, R68 to R4, R54 to R40, R62 to R41, R64 to R42, R72 to R43, R80 to R44, R82 to R45, R90 to R46, R69 to R5, R56 to R50, R57 to R51, R58 to R52, R83 to R53, R84 to R54, R85 to R55, R45 to R56, R37 to R57, R44 to R58, R3 to R59, R70 to R6, R4 to R60, R8 to R61, R9 to R62, R10 to R63, R11 to R64, R12 to R65, R13 to R66, R14 to R67, R15 to R68, R16 to R69, R77 to R7, R17 to R70, R18 to R71, R19 to R72, R20 to R73, R26 to R74, R25 to R75, R31 to R76, R23 to R77, R32 to R78, R33 to R79, R78 to R8, R5 to R80, R6 to R81, R34 to R82, R30 to R83, R27 to R84, R28 to R85, R24 to R86, R1 to R87, R2 to R88, R79 to R9, U13 to U1, U1 to U10, U3 to U11, U18 to U12, U5 to U13, U4 to U14, U19 to U15, U9 to U16, U20 to U18, U8 to U19, U14 to U2, U15 to U3, U16 to U4, U6 to U5, U10 to U6, U11 to U7, U7 to U8, U12 to U9
Connections:
- net +5V: now also J8.1 (Pin_1); no longer U1.10 (MR#), U1.16 (VCC), U2.10 (MR#), U2.16 (VCC), U3.10 (MR#), U3.16 (VCC), U4.10 (MR#), U4.16 (VCC)
- net A_VCC: now also J8.3 (Pin_3)
- new net: J8.2 (Pin_2), U1.10 (MR#), U1.16 (VCC), U2.10 (MR#), U2.16 (VCC), U3.10 (MR#), U3.16 (VCC), U4.10 (MR#), U4.16 (VCC)
Other:
- note added: "NEED BIGGER, abs max ~ 2.5A"
- note added: "Z-Interceptor"
- note added: "if feeding the 3v3, need several amps, 3a max?"
- moved on the sheet: C18, C26, C27, C28, C29, C30, U10

Commit message: add prototypes for most of BDrings modules
Parts:
- added J10, J11, J12, J13, J14, J15, J16, J17, J18, J9: Conn_01x12, symbol Connector_Generic:Conn_01x12
Connections:
- net +5V: now also J10.3 (Pin_3), J11.3 (Pin_3), J13.3 (Pin_3), J17.3 (Pin_3), J18.3 (Pin_3)
- net GND: now also J10.1 (Pin_1), J10.12 (Pin_12), J11.1 (Pin_1), J11.12 (Pin_12), J12.1 (Pin_1), J12.12 (Pin_12), J13.1 (Pin_1), J13.12 (Pin_12), J15.1 (Pin_1), J15.12 (Pin_12), J17.1 (Pin_1), J17.12 (Pin_12), J18.1 (Pin_1), J18.12 (Pin_12), J9.1 (Pin_1), J9.12 (Pin_12)
- net Vdrive: now also J12.2 (Pin_2), J13.2 (Pin_2), J9.2 (Pin_2)
- new net Inp_1_INPUT: J11.4 (Pin_4), J12.4 (Pin_4), J13.4 (Pin_4)
- new net Inp_2_INPUT: J11.5 (Pin_5), J12.5 (Pin_5), J13.5 (Pin_5)
- new net Inp_3_INPUT: J11.6 (Pin_6), J12.6 (Pin_6), J13.6 (Pin_6)
- new net Inp_4_INPUT: J11.7 (Pin_7), J13.7 (Pin_7)
- new net Mod_Ctrl_OUTPUT: J17.5 (Pin_5)
- new net Mod_Rx_INPUT: J17.6 (Pin_6)
- new net Mod_Tx_OUTPUT: J17.4 (Pin_4)
- new net OUT_1_OUTPUT: J10.7 (Pin_7), J15.7 (Pin_7), J9.5 (Pin_5)
- new net OUT_2_OUTPUT: J10.6 (Pin_6), J15.6 (Pin_6), J9.6 (Pin_6)
- new net OUT_3_OUTPUT: J10.5 (Pin_5), J15.5 (Pin_5)
- new net OUT_4_OUTPUT: J10.4 (Pin_4), J15.4 (Pin_4)
- new net Relay_OUTPUT: J18.4 (Pin_4)
- new net Spindle_DAC: J9.4 (Pin_4)
- no-connect marks 32 -> 78
Other:
- note added: "BDring 0-10V Module"
- note added: "BDring 4x_5V_Buffer_Output"
- note added: "BDring 4x_Opto_Input"
- note added: "BDring High_Current_Analog - Ths schematic looks incomplete"
- note added: "BDring Protoboard - No pdf"
- note added: "BDring Quad_Input"
- note added: "BDring Quad_MOSFET - uses external power"
- note added: "BDring RC_Servo - no PDF"
- note added: "BDring RS485"
- note added: "BDring Relay"

Commit message: add smps for 5v and 12v, add more module prototypes
Parts:
- added C32, C35: 120uF, symbol Device:C_Polarized_Small
- added C33, C34, C37: 180uF, symbol Device:C_Polarized_Small
- added C36: 220uF, symbol Device:C_Polarized_Small
- added D25, D26: 2A, 0.7V, symbol Device:D_Schottky_Small
- added J19, J20, J21: Conn_01x12, symbol Connector_Generic:Conn_01x12
- added L1, L3: 68uH, symbol Device:L_Small
- added L2, L4: 3uH, symbol Device:L_Small
- added U20: Module A4, Connector_PinSocket_2.54mm:PinSocket_1x12_P2.54mm_Vertical, symbol 111_Torban_Symbols:BDring_IO_Module
- added U21: Module A5, Connector_PinSocket_2.54mm:PinSocket_1x12_P2.54mm_Vertical, symbol 111_Torban_Symbols:BDring_IO_Module
- added U22: LM2596S-12, Package_TO_SOT_SMD:TO-263-5_TabPin3, symbol Regulator_Switching:LM2596S-12
- added U23: LM2596S-5, Package_TO_SOT_SMD:TO-263-5_TabPin3, symbol Regulator_Switching:LM2596S-5
Connections:
- net +5V: now also C37.1, L4.2
- net A_MISO: now also U20.11 (8), U21.11 (8)
- net A_MOSI: now also U20.9 (6), U21.9 (6)
- net A_SCLK: now also U20.8 (5), U21.8 (5)
- net A_VCC: now also U20.3 (VCC), U21.3 (VCC)
- net GND: now also C32.2, C33.2, C34.2, C35.2, C36.2, C37.2, D25.2 (A), D26.2 (A), J19.1 (Pin_1), J19.12 (Pin_12), J20.1 (Pin_1), J20.12 (Pin_12), J21.1 (Pin_1), J21.12 (Pin_12), U20.1 (Gnd), U20.12 (Gnd), U21.1 (Gnd), U21.12 (Gnd), U22.3 (GND), U22.5 (~{ON}/OFF), U23.3 (GND), U23.5 (~{ON}/OFF)
- net Inp_1_INPUT: now also J19.4 (Pin_4)
- net Inp_2_INPUT: now also J19.5 (Pin_5)
- net Inp_3_INPUT: now also J19.6 (Pin_6)
- net Inp_4_INPUT: now also J19.7 (Pin_7)
- net Vdrive renamed +12V
- net +12V: now also C34.1, J19.2 (Pin_2), J21.2 (Pin_2), L2.2, U20.2 (VMot), U21.2 (VMot)
- new net: D26.1 (K), L3.1, U23.2 (OUT)
- new net: C36.1, L3.2, L4.1, U23.4 (FB)
- new net: D25.1 (K), L1.1, U22.2 (OUT)
- new net: C33.1, L1.2, L2.1, U22.4 (FB)
- new net +24V: C32.1, C35.1, U22.1 (VIN), U23.1 (VIN)
- new net +3V3: J19.3 (Pin_3), J20.3 (Pin_3)
- new net Alert/Ready_INPUT: J20.9 (Pin_9)
- new net GRBL IO26 Handover: J21.4 (Pin_4)
- new net IO21 Recieve Handover: J21.9 (Pin_9)
- new net SCL: J20.11 (Pin_11)
- new net SDA: J20.10 (Pin_10)
- new net Torch IO22 Ready: J21.8 (Pin_8)
- new net Torch IO32 Trigger: J21.11 (Pin_11)
- new net Torch_IO36 THC: J21.10 (Pin_10)
- no-connect marks 78 -> 92
Other:
- note added: "120mOhm"
- note added: "16mOhm"
- note added: "18mOhm"
- note added: "24V -> 12V@3A Buck Supply"
- note added: "24V -> 5V@3A Buck Supply"
- note added: "30mOhm"
- note added: "4 Channel Screw Term"
- note added: "68mOhm"
- note added: "External A/D"
- note added: "Torch Module"
- note removed: "12V SMPS Buck Supply (24V In)"
- note removed: "5V SMPS Buck Supply"
- note removed: "if feeding the 3v3, need several amps, 3a max?"

Commit message: add leds to smps
Parts:
- added D27, D28: LED_Small_Filled, symbol Device:LED_Small_Filled
- added R89: 1K, Resistor_SMD:R_0603_1608Metric, symbol Device:R_Small
- added R90: 430R, Resistor_SMD:R_0603_1608Metric, symbol Device:R_Small
Connections:
- net +12V: now also R89.2
- net +5V: now also R90.2
- net GND: now also D27.1 (K), D28.1 (K)
- new net: D28.2 (A), R90.1
- new net: D27.2 (A), R89.1
Other:
- moved on the sheet: C26, C27, C28, C29, C30

Commit message: redesigned 5v psu to more modern chip. start working on lcsc pn's
Parts:
- removed C35: 120uF, symbol Device:C_Polarized_Small
- removed C36: 220uF, symbol Device:C_Polarized_Small
- removed C37: 180uF, symbol Device:C_Polarized_Small
- removed D26: 2A, 0.7V, symbol Device:D_Schottky_Small
- removed D28: LED_Small_Filled, symbol Device:LED_Small_Filled
- removed L3: 68uH, symbol Device:L_Small
- removed L4: 3uH, symbol Device:L_Small
- removed R90: 430R, Resistor_SMD:R_0603_1608Metric, symbol Device:R_Small
- removed U23: LM2596S-5, Package_TO_SOT_SMD:TO-263-5_TabPin3, symbol Regulator_Switching:LM2596S-5
- added C31, C42: 10nF, Capacitor_SMD:C_0603_1608Metric, symbol Device:C_Small
- added C38, C40, C41: 10uF, Capacitor_SMD:C_0805_2012Metric, symbol Device:C_Small
- added C39: 330uF, Capacitor_Tantalum_SMD:CP_EIA-7343-31_Kemet-D, symbol Device:C_Polarized_Small
- added D29: SS54, Diode_SMD:D_SMA, symbol Device:D_Schottky_Small
- added D30: Emerald, LED_SMD:LED_0603_1608Metric, symbol Device:LED_Small_Filled
- added L5: 15uH, Inductor_SMD:L_Sunlord_MWSA0603S, symbol Device:L_Small
- added R91: 10K, Resistor_SMD:R_0603_1608Metric, symbol Device:R_Small
- added R92: 3.24K, Resistor_SMD:R_0603_1608Metric, symbol Device:R_Small
- added R93: 430R, Resistor_SMD:R_0603_1608Metric, symbol Device:R_Small
- added U24: TPS5430DDA, Package_SO:TI_SO-PowerPAD-8_ThermalVias, symbol Regulator_Switching:TPS5430DDA
- D1, D10, D11, D12, D13, D14, D15, D16, D17, D18, D2, D21, D22, D27, D3, D4, D5, D6, D7, D8, D9: value LED_Small_Filled -> Emerald; footprint (none) -> LED_SMD:LED_0603_1608Metric; LCSC (none) -> C72043
- H1, J2, JP1, JP2, JP5, JP6, U11, U12, U14, U15, U17, U18, U20, U21: LCSC (none) -> DNP
- R1, R2, R29, R3, R30, R31, R32, R33, R34, R35, R36, R37, R4, R5, R6, R7, R8, R9: LCSC (none) -> C8218
- R10, R11, R12, R13, R14, R15, R16, R17, R18, R38, R39, R40, R41, R42, R43, R44, R45, R46, R89: LCSC (none) -> C21190
- R19, R20, R21, R22, R23, R24, R25, R26, R27, R28, R47, R48, R49, R50, R51, R52, R53, R54, R55, R80, R81, R83, R87, R88: LCSC (none) -> C25804
- R56, R57, R58, R59, R60, R61, R62, R63, R64, R65, R66, R67, R68, R69, R70, R71, R72, R73: value 500R -> 510R; LCSC (none) -> C23193
- R74, R75, R84, R85: LCSC (none) -> C23186
- R76, R79: LCSC (none) -> C25803
- R77, R86: LCSC (none) -> C23162
- R78, R82: LCSC (none) -> C23159
- U22: LCSC (none) -> C2980821
Connections:
- net +24V: now also C38.1, C40.1, C41.1, U24.7 (VIN)
- net +5V: now also C39.1, L5.2, R91.2, R93.2
- net GND: now also C38.2, C39.2, C40.2, C41.2, D29.2 (A), D30.1 (K), R92.1, U24.6 (GND), U24.9 (GNDPAD)
- new net: C42.1, U24.1 (BOOT)
- new net: R91.1, R92.2, U24.4 (VSENSE)
- new net: C42.2, D29.1 (K), L5.1, U24.8 (PH)
- new net: D30.2 (A), R93.1
- no-connect marks 92 -> 93
Other:
- note removed: "120mOhm"
- note removed: "68mOhm"
- moved on the sheet: C32, C33, C34, D25, D27, L1, L2, R89, U22
