File: Hardware/Main Board V2.0/Main Board/Main Board.kicad_sch (KiCad schematic)
At the start: 241 parts, among them J10 Conn_01x12, J11 Conn_01x12, J12 Conn_01x12, J13 Conn_01x12, J14 Conn_01x12, J15 Conn_01x12, J16 Conn_01x12, J16 Micro_SD_Card, J17 Conn_01x12, J18 Conn_01x12, J19 Conn_01x12, J2 Screw_Terminal_01x06, J20 Conn_01x12, J21 Conn_01x12, J8 Conn_01x03, J9 Conn_01x12, Q1 BSS138, Q19 MMBT2222, Q20 MMBT2222, Q21 MMBT2222, Q22 MMBT2222, SW1 SW_Push, SW2 SW_Push, U1 74AHCT595PW, U10 74LVC157A, U11 Module A1, U12 Module B1, U13 ESP32-WROOM-32UE-H4, U14 Module A2, U15 Module B2, U16 GT-USB-7051A, U17 Module A3, U18 Module B3, U19 CP2104, U2 74AHCT595PW, U20 Module A4, U21 Module A5, U22 LM2596S-12, U23 AP2112K-3.3, U24 TPS5430DDA, U25 AP2112K-3.3, U3 74AHCT595PW, U4 74AHCT595PW, U5 ESP32-WROOM-32UE-H4, U6 GT-USB-7051A, U8 CP2104

Commit message: create a generic reference design for modules
Parts:
- added J22, J23: Conn_01x12, symbol Connector_Generic:Conn_01x12
Connections:
- net +5V is gone; now on net +12V: C35.1, C39.1, C4.1, C43.1, C5.1, C6.1, C7.1, J10.3 (Pin_3), J11.3 (Pin_3), J13.3 (Pin_3), J17.3 (Pin_3), J18.3 (Pin_3), J8.1 (Pin_1), L5.2, R90.2, R91.2, R93.2, R95.2, U23.1 (VIN), U25.1 (VIN)
- net +12V: now also C1.1, C10.2, C11.2, C12.2, C14.2, C18.2, C19.1, C2.2, C20.2, C21.2, C22.2, C23.2, C24.2, C25.1, C3.2, C32.2, C35.2, C36.2, C37.2, C38.2, C39.2, C4.2, C40.2, C41.2, C43.2, C44.2, C45.2, C5.2, C6.2, C7.2, C8.2, C9.2, D20.1 (VN), D24.1 (VN), D25.2 (A), D26.1 (K), D27.1 (K), D28.1 (K), D29.2 (A), D30.1 (K), H1.1, H1.1, H1.1, H1.1, H1.1, H1.1, H1.1, J10.1 (Pin_1), J10.2 (Pin_2), J11.1 (Pin_1), J11.2 (Pin_2), J12.1 (Pin_1), J12.3 (Pin_3), J13.1 (Pin_1), J15.1 (Pin_1), J15.2 (Pin_2), J15.3 (Pin_3), J16.6 (VSS), J16.9 (SHIELD), J17.1 (Pin_1), J17.2 (Pin_2), J18.1 (Pin_1), J18.2 (Pin_2), J19.1 (Pin_1), J19.12 (Pin_12), J20.1 (Pin_1), J20.12 (Pin_12), J21.1 (Pin_1), J21.12 (Pin_12), J9.1 (Pin_1), J9.3 (Pin_3), Q1.2 (S), Q1.2 (S), Q1.2 (S), Q1.2 (S), Q1.2 (S), Q1.2 (S), Q1.2 (S), Q1.2 (S), Q1.2 (S), Q1.2 (S), Q1.2 (S), Q1.2 (S), Q1.2 (S), Q1.2 (S), Q1.2 (S), Q1.2 (S), Q1.2 (S), Q1.2 (S), R19.1, R20.1, R21.1, R22.1, R23.1, R24.1, R25.1, R26.1, R27.1, R47.1, R48.1, R49.1, R50.1, R51.1, R52.1, R53.1, R54.1, R55.1, R74.1, R75.1, R84.1, R85.1, R92.1, SW1.1, SW2.1, U1.13 (OE#), U1.8 (GND), U10.15 (~{EN}), U10.8 (GND), U11.1 (Gnd), U11.12 (Gnd), U12.1 (Gnd), U12.12 (Gnd), U13.1 (GND), U13.15 (GND), U13.38 (GND), U13.39 (GND_THERMAL), U14.1 (Gnd), U14.12 (Gnd), U15.1 (Gnd), U15.12 (Gnd), U16.A1 (GND), U16.A12 (GND), U16.B1 (GND), U16.B12 (GND), U17.1 (Gnd), U17.12 (Gnd), U18.1 (Gnd), U18.12 (Gnd), U19.2 (GND), U19.25 (GND), U2.13 (OE#), U2.8 (GND), U20.1 (Gnd), U20.12 (Gnd), U21.1 (Gnd), U21.12 (Gnd), U22.3 (GND), U22.5 (~{ON}/OFF), U23.2 (GND), U24.6 (GND), U24.9 (GNDPAD), U25.2 (GND), U3.13 (OE#), U3.8 (GND), U4.13 (OE#), U4.8 (GND), U5.1 (GND), U5.15 (GND), U5.38 (GND), U5.39 (GND_THERMAL), U6.A1 (GND), U6.A12 (GND), U6.B1 (GND), U6.B12 (GND), U8.2 (GND), U8.25 (GND), J22.1 (Pin_1), J22.12 (Pin_12), J22.2 (Pin_2), J23.1 (Pin_1), J23.12 (Pin_12), J23.2 (Pin_2), J23.3 (Pin_3)
- net OUT_1_OUTPUT: now also J22.4 (Pin_4)
- net OUT_2_OUTPUT: now also J22.5 (Pin_5)
- net OUT_3_OUTPUT: now also J22.6 (Pin_6)
- net OUT_4_OUTPUT: now also J22.7 (Pin_7)
- removed net GND: C1.1, C10.2, C11.2, C12.2, C14.2, C18.2, C19.1, C2.2, C20.2, C21.2, C22.2, C23.2, C24.2, C25.1, C3.2, C32.2, C35.2, C36.2, C37.2, C38.2, C39.2, C4.2, C40.2, C41.2, C43.2, C44.2, C45.2, C5.2, C6.2, C7.2, C8.2, C9.2, D20.1 (VN), D24.1 (VN), D25.2 (A), D26.1 (K), D27.1 (K), D28.1 (K), D29.2 (A), D30.1 (K), H1.1, H1.1, H1.1, H1.1, H1.1, H1.1, H1.1, J10.1 (Pin_1), J10.12 (Pin_12), J11.1 (Pin_1), J11.12 (Pin_12), J12.1 (Pin_1), J12.12 (Pin_12), J13.1 (Pin_1), J13.12 (Pin_12), J15.1 (Pin_1), J15.12 (Pin_12), J16.6 (VSS), J16.9 (SHIELD), J17.1 (Pin_1), J17.12 (Pin_12), J18.1 (Pin_1), J18.12 (Pin_12), J19.1 (Pin_1), J19.12 (Pin_12), J20.1 (Pin_1), J20.12 (Pin_12), J21.1 (Pin_1), J21.12 (Pin_12), J9.1 (Pin_1), J9.12 (Pin_12), Q1.2 (S), Q1.2 (S), Q1.2 (S), Q1.2 (S), Q1.2 (S), Q1.2 (S), Q1.2 (S), Q1.2 (S), Q1.2 (S), Q1.2 (S), Q1.2 (S), Q1.2 (S), Q1.2 (S), Q1.2 (S), Q1.2 (S), Q1.2 (S), Q1.2 (S), Q1.2 (S), R19.1, R20.1, R21.1, R22.1, R23.1, R24.1, R25.1, R26.1, R27.1, R47.1, R48.1, R49.1, R50.1, R51.1, R52.1, R53.1, R54.1, R55.1, R74.1, R75.1, R84.1, R85.1, R92.1, SW1.1, SW2.1, U1.13 (OE#), U1.8 (GND), U10.15 (~{EN}), U10.8 (GND), U11.1 (Gnd), U11.12 (Gnd), U12.1 (Gnd), U12.12 (Gnd), U13.1 (GND), U13.15 (GND), U13.38 (GND), U13.39 (GND_THERMAL), U14.1 (Gnd), U14.12 (Gnd), U15.1 (Gnd), U15.12 (Gnd), U16.A1 (GND), U16.A12 (GND), U16.B1 (GND), U16.B12 (GND), U17.1 (Gnd), U17.12 (Gnd), U18.1 (Gnd), U18.12 (Gnd), U19.2 (GND), U19.25 (GND), U2.13 (OE#), U2.8 (GND), U20.1 (Gnd), U20.12 (Gnd), U21.1 (Gnd), U21.12 (Gnd), U22.3 (GND), U22.5 (~{ON}/OFF), U23.2 (GND), U24.6 (GND), U24.9 (GNDPAD), U25.2 (GND), U3.13 (OE#), U3.8 (GND), U4.13 (OE#), U4.8 (GND), U5.1 (GND), U5.15 (GND), U5.38 (GND), U5.39 (GND_THERMAL), U6.A1 (GND), U6.A12 (GND), U6.B1 (GND), U6.B12 (GND), U8.2 (GND), U8.25 (GND)
- new net GPIO OR ADC+: J23.6 (Pin_6)
- new net GPIO OR ADC-: J23.7 (Pin_7)
- new net GPIO OR DAC: J23.4 (Pin_4)
- new net GPIO OR PWM: J23.5 (Pin_5)
- new net SPI_CS OR I2C_SDA: J23.10 (Pin_10)
- new net SPI_MISO OR I2C_SCL: J23.11 (Pin_11)
- new net SPI_MOSI OR GPIO: J23.9 (Pin_9)
- new net SPI_SCLK OR GPIO: J23.8 (Pin_8)
- no-connect marks 93 -> 98
Other:
- note added: "Generic Reference Design"
- note added: "Quad Output Module"
- note added: "Torch mudule likely needs redesign"
- moved on the sheet: C11, C32, C8, D25, D27, J10, J11, J12, J13, J14, J15, J16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

Commit message: designing expansion modules
Parts:
- removed U14: Module A2, Connector_PinSocket_2.54mm:PinSocket_1x12_P2.54mm_Vertical, symbol 111_Torban_Symbols:BDring_IO_Module
- removed U15: Module B2, Connector_PinSocket_2.54mm:PinSocket_1x12_P2.54mm_Vertical, symbol 111_Torban_Symbols:BDring_IO_Module
- removed U18: Module B3, Connector_PinSocket_2.54mm:PinSocket_1x12_P2.54mm_Vertical, symbol 111_Torban_Symbols:BDring_IO_Module
- removed U21: Module A5, Connector_PinSocket_2.54mm:PinSocket_1x12_P2.54mm_Vertical, symbol 111_Torban_Symbols:BDring_IO_Module
- added SW10, SW3, SW4, SW5, SW6, SW7, SW8, SW9: SW_DPDT_x2, symbol Switch:SW_DPDT_x2
- added U16: Module A2, Connector_PinSocket_2.54mm:PinSocket_1x12_P2.54mm_Vertical, symbol 111_Torban_Symbols:BDring_IO_Module
- added U19: Module A3, Connector_PinSocket_2.54mm:PinSocket_1x12_P2.54mm_Vertical, symbol 111_Torban_Symbols:BDring_IO_Module
- added U22: Module A4, Connector_PinSocket_2.54mm:PinSocket_1x12_P2.54mm_Vertical, symbol 111_Torban_Symbols:BDring_IO_Module
- added U23: Module B4, Connector_PinSocket_2.54mm:PinSocket_1x12_P2.54mm_Vertical, symbol 111_Torban_Symbols:BDring_IO_Module
- U17: value Module A3 -> Module B2
- U20: value Module A4 -> Module B3
- renumbered C35 to C10, C10 to C11, C41 to C12, C12 to C13, C40 to C14, C36 to C15, C14 to C16, C38 to C17, C37 to C18, C8 to C19, C11 to C20, C42 to C21, C43 to C22, C39 to C23, C44 to C24, C45 to C25, C18 to C26, C19 to C27, C20 to C28, C21 to C29, C22 to C30, C23 to C31, C24 to C32, C25 to C33, C26 to C34, C27 to C35, C28 to C36, C29 to C37, C30 to C38, C31 to C39, C32 to C8, D25 to D20, D20 to D21, D26 to D22, D27 to D23, D29 to D24, D30 to D25, D28 to D26, D23 to D27, D24 to D28, J19 to J10, J23 to J11, J10 to J12, J20 to J13, J11 to J14, J21 to J15, J12 to J16, J22 to J17, J13 to J18, J14 to J19, J15 to J20, J16 to J21, J17 to J22, J18 to J23, JP5 to JP3, JP6 to JP4, L5 to L3, R90 to R76, R94 to R78, R89 to R79, R95 to R82, R91 to R83, R92 to R84, R93 to R85, R96 to R86, R83 to R87, R84 to R88, R85 to R89, R86 to R90, R87 to R91, R88 to R92, U24 to U10, U25 to U11, U10 to U12, U11 to U13, U12 to U14, U13 to U15, U16 to U18, U19 to U21, U22 to U7, U23 to U8, U8 to U9
Connections:
- net +12V: now also U13.3 (VCC), U14.3 (VCC), U17.3 (VCC), U20.3 (VCC), U16.1 (Gnd), U16.12 (Gnd), U16.2 (VMot), U16.3 (VCC), U19.1 (Gnd), U19.12 (Gnd), U19.2 (VMot), U19.3 (VCC), U22.1 (Gnd), U22.12 (Gnd), U22.2 (VMot), U22.3 (VCC), U23.1 (Gnd), U23.12 (Gnd), U23.2 (VMot), U23.3 (VCC)
- net A_MISO: now also SW3.1 (A), SW5.1 (A), SW7.1 (A), SW9.1 (A); no longer U13.11 (8), U17.11 (8), U20.11 (8)
- net A_MOSI: now also U16.9 (6), U19.9 (6), U22.9 (6); no longer U17.9 (6), U20.9 (6)
- net A_SCL: now also SW3.3 (C), SW5.3 (C), SW7.3 (C), SW9.3 (C)
- net A_SCLK: now also U16.8 (5), U19.8 (5), U22.8 (5); no longer U17.8 (5), U20.8 (5)
- net A_SDA: now also SW3.6 (C), SW5.6 (C), SW7.6 (C), SW9.6 (C)
- net A_VCC: no longer U13.3 (VCC), U17.3 (VCC), U20.3 (VCC)
- net B_MISO: now also SW10.1 (A), SW4.1 (A), SW6.1 (A), SW8.1 (A); no longer U14.11 (8)
- net B_MOSI: now also U17.9 (6), U20.9 (6), U23.9 (6)
- net B_SCL: now also SW10.3 (C), SW4.3 (C), SW6.3 (C), SW8.3 (C)
- net B_SCLK: now also U17.8 (5), U20.8 (5), U23.8 (5)
- net B_SDA: now also SW10.6 (C), SW4.6 (C), SW6.6 (C), SW8.6 (C)
- net B_VCC: no longer U14.3 (VCC)
- net at U17.10 (7): now also SW6.5 (B)
- net at U13.10 (7): now also SW3.5 (B)
- net at U14.10 (7): now also SW4.5 (B)
- net at U20.10 (7): now also SW8.5 (B)
- new net: SW5.5 (B), U16.10 (7)
- new net: SW5.2 (B), U16.11 (8)
- new net: SW3.2 (B), U13.11 (8)
- new net: SW10.5 (B), U23.10 (7)
- new net: SW10.2 (B), U23.11 (8)
- new net: SW4.2 (B), U14.11 (8)
- new net: SW6.2 (B), U17.11 (8)
- new net: SW9.2 (B), U22.11 (8)
- new net: SW7.5 (B), U19.10 (7)
- new net: SW7.2 (B), U19.11 (8)
- new net: SW8.2 (B), U20.11 (8)
- new net: SW9.5 (B), U22.10 (7)
Other:
- note added: "TODO - Find replacement for this archaic part"
- moved on the sheet: U13, U14

Commit message: updated comments for further changes, add uart
Parts:
- removed U23: Module B4, Connector_PinSocket_2.54mm:PinSocket_1x12_P2.54mm_Vertical, symbol 111_Torban_Symbols:BDring_IO_Module
- added D29: D_Schottky, symbol Device:D_Schottky
- added SW11: SW_DPDT_x2, symbol Switch:SW_DPDT_x2
Connections:
- net A_MOSI: now also SW10.3 (C); no longer U13.9 (6)
- net A_SCLK: now also SW10.6 (C); no longer U13.8 (5)
- net B_GPIO_19: now also U15.31 (GPIO19)
- net B_MISO: no longer SW10.1 (A)
- net B_MOSI: now also SW11.3 (C); no longer U14.9 (6)
- net B_SCL: no longer SW10.3 (C)
- net B_SCLK: now also SW11.6 (C); no longer U14.8 (5)
- net B_SDA: no longer SW10.6 (C)
- net at SW10.5 (B): now also U13.8 (5)
- net at SW10.2 (B): now also U13.9 (6)
- net B_GPIO_16 renamed B_RX2
- net B_RX2: now also SW11.4 (A)
- net B_GPIO_17 renamed B_TX2
- net B_TX2: now also SW11.1 (A)
- net Z_Enable_THC: no longer names the net of U12.3 (I1a)
- net Z_Enable_THC: no longer U15.31 (GPIO19)
- new net: SW11.5 (B), U14.8 (5)
- new net: SW11.2 (B), U14.9 (6)
Other:
- note added: "Notes: - ESP32 with antenna only available with 4mb flash at jlcpcb. which should work with fluidnc - TODO - reset brought out - jtag - usb to power other things? jumper? - i2c pullups - nextion display? on a module? uart? - general purpose inputs may need pull up and down - joining pins --- gpio hold (input to fluidnc) (want it to shit of plasma torch) --- gpio start (input to fluidnc) --- gpio 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"
- note added: "uart???"
- note removed: "Notes: - ESP32 with antenna only available with 4mb flash at jlcpcb. which should work with fluidnc -"
- moved on the sheet: SW4A, SW4B, SW6A, SW6B, SW8A, SW8B, U14, U17, U20
