File: Hardware/Main Board V2.0/Main Board/Main Board.kicad_sch (KiCad schematic)
At the start: 252 parts, among them J10 Conn_01x12, J11 Conn_01x12, J12 Conn_01x12, J13 Conn_01x12, J14 Conn_01x12, J15 Conn_01x12, J16 Conn_01x12, J16 Micro_SD_Card, J17 Conn_01x12, J18 Conn_01x12, J19 Conn_01x12, J2 Screw_Terminal_01x06, J20 Conn_01x12, J21 Conn_01x12, J22 Conn_01x12, J23 Conn_01x12, J8 Conn_01x03, J9 Conn_01x12, Q1 BSS138, Q19 MMBT2222, Q20 MMBT2222, Q21 MMBT2222, Q22 MMBT2222, SW1 SW_Push, SW10 SW_DPDT_x2, SW11 SW_DPDT_x2, SW2 SW_Push, SW3 SW_DPDT_x2, SW4 SW_DPDT_x2, SW5 SW_DPDT_x2, SW6 SW_DPDT_x2, SW7 SW_DPDT_x2, SW8 SW_DPDT_x2, SW9 SW_DPDT_x2, U1 74AHCT595PW, U10 TPS5430DDA, U11 AP2112K-3.3, U12 74LVC157A, U13 Module A1, U14 Module B1, U15 ESP32-WROOM-32UE-H4, U16 Module A2, U17 Module B2, U18 GT-USB-7051A, U19 Module A3, U2 74AHCT595PW, U20 Module B3, U21 CP2104, U22 Module A4, U3 74AHCT595PW, U4 74AHCT595PW, U5 ESP32-WROOM-32UE-H4, U6 GT-USB-7051A, U7 LM2596S-12, U8 AP2112K-3.3, U9 CP2104

Commit message: v2 work
Parts:
- removed C27, C31: 1uF, Capacitor_SMD:C_0805_2012Metric, symbol Device:C_Small
- removed C28: 22uF, Capacitor_SMD:C_1206_3216Metric, symbol Device:C_Small
- removed C29, C32: 100nF, Capacitor_SMD:C_0603_1608Metric, symbol Device:C_Small
- removed C30, C33: 4.7uF, Capacitor_SMD:C_0805_2012Metric, symbol Device:C_Small
- removed D26: Emerald, LED_SMD:LED_0603_1608Metric, symbol Device:LED_Small_Filled
- removed D27: D_Schottky, symbol Device:D_Schottky
- removed D28: SP0503BAHT, Package_TO_SOT_SMD_AKL:SOT-143, symbol PCM_Diode_TVS_AKL:SP0503BAHT
- removed J11: Conn_01x12, symbol Connector_Generic:Conn_01x12
- removed J2 (x6): Screw_Terminal_01x06, User Library:2x3 screw terminal3.5mm, symbol Connector:Screw_Terminal_01x06
- removed J8: Conn_01x03, symbol Connector_Generic:Conn_01x03
- removed JP3, JP4: SolderJumper_2_Bridged, Jumper:SolderJumper-2_P1.3mm_Bridged_RoundedPad1.0x1.5mm, symbol Jumper:SolderJumper_2_Bridged
- removed Q1 (x18): BSS138, Package_TO_SOT_SMD:SOT-23, symbol Device:Q_NMOS_GSD
- removed Q21, Q22: MMBT2222, Package_TO_SOT_SMD_AKL:SOT-23, symbol PCM_Transistor_BJT_AKL:MMBT2222
- removed R24, R87, R91, R92: 10K, Resistor_SMD:R_0603_1608Metric, symbol Device:R_Small
- removed R4: 200R, Resistor_SMD:R_0603_1608Metric, symbol Device:R_Small
- removed R88, R89: 5.1K, Resistor_SMD:R_0603_1608Metric, symbol Device:R_Small
- removed R90: 4.7K, Resistor_SMD:R_0603_1608Metric, symbol Device:R_Small
- removed SW10, SW11, SW3, SW4, SW5, SW6, SW7, SW8, SW9: SW_DPDT_x2, symbol Switch:SW_DPDT_x2
- removed SW2: SW_Push, symbol Switch:SW_Push
- removed U11: AP2112K-3.3, Package_TO_SOT_SMD:SOT-23-5, symbol Regulator_Linear:AP2112K-3.3
- removed U14: Module B1, Connector_PinSocket_2.54mm:PinSocket_1x12_P2.54mm_Vertical, symbol 111_Torban_Symbols:BDring_IO_Module
- removed U15: ESP32-WROOM-32UE-H4, Espressif:ESP32-WROOM-32UE, symbol Espressif:ESP32-WROOM-E
- removed U17: Module B2, Connector_PinSocket_2.54mm:PinSocket_1x12_P2.54mm_Vertical, symbol 111_Torban_Symbols:BDring_IO_Module
- removed U18: GT-USB-7051A, KiCad:GT-USB-7051A, symbol 111_Torban_Symbols:GT-USB-7051A
- removed U20: Module B3, Connector_PinSocket_2.54mm:PinSocket_1x12_P2.54mm_Vertical, symbol 111_Torban_Symbols:BDring_IO_Module
- removed U21: CP2104, Package_DFN_QFN:QFN-24-1EP_4x4mm_P0.5mm_EP2.6x2.6mm, symbol Interface_USB:CP2104
- added C3: 22nf, Capacitor_SMD:C_0603_1608Metric_Pad1.08x0.95mm_HandSolder, symbol Device:C_Small
- added C40: 100nF, Capacitor_SMD:C_0603_1608Metric, symbol Device:C_Small
- added C6, C8: 1uf, Capacitor_SMD:C_0603_1608Metric_Pad1.08x0.95mm_HandSolder, symbol Device:C_Small
- added C7: 100nf, Capacitor_SMD:C_0603_1608Metric_Pad1.08x0.95mm_HandSolder, symbol Device:C_Small
- added D2, D3: MSCD104H, Diode_SMD:D_0805_2012Metric_Pad1.15x1.40mm_HandSolder, symbol Device:D_Schottky_Small
- added D26, D30, D38: D_Small, symbol Device:D_Small
- added D31, D32, D33, D34, D35: Emerald, LED_SMD:LED_0603_1608Metric, symbol Device:LED_Small_Filled
- added D36, D37, D39: PESD12VL1BA, Diode_SMD_AKL:D_SOD-323_TVS, symbol PCM_Diode_TVS_AKL:PESD12VL1BA
- added FB1, FB2: BLM18HE152SN1D, Resistor_SMD:R_0603_1608Metric_Pad0.98x0.95mm_HandSolder, symbol Torch-Module-rescue:Ferrite_Bead_Small-Device
- added J12: Conn_01x02_Male, Connector_PinHeader_2.54mm:PinHeader_1x02_P2.54mm_Vertical, symbol Connector:Conn_01x02_Male
- added J15: Module conn, Connector_PinHeader_2.54mm:PinHeader_1x12_P2.54mm_Vertical, symbol Connector:Conn_01x12_Male
- added J2, J25, J3, J31, J32, J33, J34, J35, J36, J37, J38, J4, J41, J42, J43, J44, J45, J46, J47, J48, J49, J50, J51, J52, J6, J7: Conn_01x03, symbol Connector_Generic:Conn_01x03
- added J24, J26, J27, J28, J29, J30, J39: Conn_02x03_Top_Bottom, KiCad:DB2ERH-2.5-2-3P-GN, symbol Connector_Generic:Conn_02x03_Top_Bottom
- added J40, J5, J8: Conn_02x08_Top_Bottom, KiCad:DB2ERH-2.5-2-8P-GN, symbol Connector_Generic:Conn_02x08_Top_Bottom
- added K1, K2, K3: G2RL-1-E-DC12, Relay_THT:Relay_SPDT_Schrack-RT1-16A-FormC_RM5mm, symbol Relay:RT314A12
- added R105, R106, R107, R108, R109, R110, R111, R112, R113: 510R, Resistor_SMD:R_0603_1608Metric, symbol Device:R_Small
- added R114, R115, R116, R117, R119, R120, R121, R122, R123, R124, R125, R126, R127, R128, R129, R130, R131: 10K, Resistor_SMD:R_0603_1608Metric, symbol Device:R_Small
- added R118: 5K, Resistor_SMD:R_0603_1608Metric, symbol Device:R_Small
- added R30, R32, R33: 1K, Resistor_SMD:R_0603_1608Metric_Pad0.98x0.95mm_HandSolder, symbol Device:R_US
- added R31: 2K, Resistor_SMD:R_0603_1608Metric_Pad0.98x0.95mm_HandSolder, symbol Device:R_US
- added R34, R35, R36, R37: 2.4K, Resistor_SMD:R_0603_1608Metric_Pad0.98x0.95mm_HandSolder, symbol Device:R_US
- added R38, R39: 200, Resistor_SMD:R_0603_1608Metric_Pad0.98x0.95mm_HandSolder, symbol Device:R_US
- added R4 (x12): 2K, Resistor_SMD:R_0603_1608Metric_Pad0.98x0.95mm_HandSolder, symbol Device:R_Small
- added R4: 1K, Resistor_SMD:R_0603_1608Metric, symbol Device:R_Small
- added RV1, RV2: 20K, symbol Device:R_Potentiometer
- added SW12: SW_Push, symbol Switch:SW_Push
- added U2: NCV8114ASN150T1G, Package_TO_SOT_SMD:TSOT-23-5, symbol Regulator_Linear:NCV8114ASN150T1G
- added U23: XTSD04GLGEAG, KiCad:SON127P600X800X95-8N, symbol 111_Torban_Symbols:XTSD04GLGEAG
- added U24, U25, U26: ELQ3H7, KiCad:ELQ3H7 SOP-16_4.4x10.4mm_P1.27mm, symbol Isolator:LTV-847S
- added U29: MAX3485, symbol Interface_UART:MAX3485
- added U3 (x3): ULN2003A, Package_SO:SOIC-16_3.9x9.9mm_P1.27mm, symbol Transistor_Array:ULN2003A
- added U3: ADS1115IDGS, Package_SO:TSSOP-10_3x3mm_P0.5mm, symbol Analog_ADC:ADS1115IDGS
- added U30: LM358, symbol Amplifier_Operational:LM358
- C1, C25: value 1uF -> 100nF; footprint Capacitor_SMD:C_0805_2012Metric -> Capacitor_SMD:C_0603_1608Metric; LCSC C28323 -> C14663
- C22, C24: value 10uF -> 100nF; footprint Capacitor_SMD:C_0805_2012Metric -> Capacitor_SMD:C_0603_1608Metric; LCSC C440198 -> C14663
- J16: now not fitted
- R1, R2, R3, R5, R6, R7, R8, R9: value 200R -> 1K; LCSC C8218 -> C21190
- R19, R20, R21, R50, R51: value 10K -> 1K; LCSC C25804 -> C21190
- R23, R54: value 10K -> 20R; LCSC C25804 -> C21190
- R25: value 10K -> 120R; LCSC C25804 -> (none)
- R26: value 10K -> 24K; LCSC C25804 -> (none)
- R27: value 10K -> 47K; LCSC C25804 -> (none)
- R29, R30, R31, R32, R33, R34, R35, R36, R37: value 200R -> 10K; LCSC C8218 -> C25804
- R38, R39, R40, R41, R42, R43, R44, R45, R46: value 1K -> 10K; LCSC C21190 -> C25804
- R71, R72: value 510R -> 10K; LCSC C23193 -> C25804
- R73: value 510R -> 5K; LCSC C23193 -> C21190
- R82: value 100K -> 10K; LCSC C25803 -> C25804
- R86: value 4.3K -> 10K; LCSC C23159 -> C25804
- U5: footprint Espressif:ESP32-WROOM-32UE -> KiCad:ESP32-WROOM-32UE
Connections:
- net A_GPIO_18 is gone; now on net SDA: U5.30 (GPIO18)
- net A_GPIO_19 is gone; now on net SCL: U5.31 (GPIO19)
- net A_GPIO_2 is gone; now on net PWM1: U5.24 (ADC2_CH2/GPIO2)
- net A_GPIO_23 is gone; now on net I2S_BCK: U5.37 (GPIO23)
- net A_VCC is gone; now on net +3V3: C11.1, C13.1, C15.1, C18.1, C2.1, C3.1, C9.1, J16.4 (VDD), R28.2, R77.2, R78.2, U5.2 (3V3), U8.5 (VOUT), U9.5 (VIO), U9.6 (VDD), U9.7 (REGIN)
- net Z_Enable_GRBL is gone; now on net Z_Enable: U12.2 (I0a), U2.15 (Q0)
- net +12V: now also C1.2, C26.1, R1.2, R19.2, R2.2, R20.2, R21.2, R29.1, R3.2, R30.1, R31.1, R32.1, R33.1, R34.1, R35.1, R36.1, R37.1, R38.1, R39.1, R40.1, R41.1, R42.1, R43.1, R44.1, R45.1, R46.1, R5.2, R6.2, R7.2, R8.2, R9.2, U1.10 (MR#), U1.16 (VCC), U12.16 (VCC), U2.10 (MR#), U2.16 (VCC), U3.10 (MR#), U3.16 (VCC), U4.10 (MR#), U4.16 (VCC), C40.2, D26.2 (A), D30.2 (A), D37.2 (A), D38.2 (A), J2.1 (Pin_1), J2.3 (Pin_3), J24.3 (Pin_3), J24.6 (Pin_6), J25.1 (Pin_1), J26.1 (Pin_1), J26.3 (Pin_3), J26.4 (Pin_4), J26.6 (Pin_6), J27.1 (Pin_1), J27.3 (Pin_3), J27.4 (Pin_4), J27.6 (Pin_6), J28.1 (Pin_1), J28.3 (Pin_3), J28.4 (Pin_4), J28.6 (Pin_6), J29.1 (Pin_1), J29.3 (Pin_3), J29.4 (Pin_4), J29.6 (Pin_6), J3.1 (Pin_1), J3.3 (Pin_3), J30.1 (Pin_1), J30.3 (Pin_3), J30.4 (Pin_4), J30.6 (Pin_6), J33.1 (Pin_1), J33.3 (Pin_3), J36.1 (Pin_1), J39.1 (Pin_1), J39.3 (Pin_3), J39.4 (Pin_4), J39.6 (Pin_6), J4.1 (Pin_1), J4.3 (Pin_3), J43.1 (Pin_1), J48.1 (Pin_1), J6.1 (Pin_1), J6.3 (Pin_3), J7.1 (Pin_1), J7.3 (Pin_3), K1.A2, K2.A2, K3.A2, R114.1, R115.1, R117.2, R119.1, R4.1, R4.1, R4.1, R4.1, R4.1, R4.1, R4.1, R4.1, R4.1, R4.1, R4.1, R4.1, R4.2, SW12.1, U23.4 (VSS), U24.11, U24.13, U24.15, U24.9, U25.11, U25.13, U25.15, U25.9, U26.11, U26.13, U26.15, U26.9, U29.5 (GND), U3.8 (GND), U3.8 (GND), U3.8 (GND), U3.9 (COM), U3.9 (COM), U3.9 (COM), U30.4 (V-), U30.8 (V+); no longer C1.1, C22.1, R19.1, R20.1, R21.1, R22.1, R23.1, R25.1, R26.1, R38.2, R39.2, R40.2, R41.2, R42.2, R43.2, R44.2, R45.2, R46.2, R50.1, R51.1, R52.1, R54.1, R55.1, R56.1, R57.1, R58.1, R59.1, R60.1, R61.1, R62.1, R63.1, R64.1, R65.1, R66.1, R67.1, R68.1, R69.1, R70.1, R71.1, R72.1, R73.1, U13.3 (VCC), U16.3 (VCC), U19.3 (VCC), U22.3 (VCC)
- net +3V3: now also C22.1, R22.2, R50.2, R51.2, R52.2, R55.2, R71.2, R72.2, D36.2 (A), J25.3 (Pin_3), J36.3 (Pin_3), J43.3 (Pin_3), J48.3 (Pin_3), R120.1, R121.1, R122.1, R123.1, R124.1, R125.1, R126.1, R127.1, R128.1, R129.1, R130.1, R131.1, U23.8 (VDD), U29.8 (VCC)
- net A_Dir: now also R37.2, U3.6 (I6); no longer R31.2
- net A_Dir_HV: now also D13.1 (K), J40.13 (Pin_13), U3.11 (O6); no longer D12.1 (K)
- net A_Enable: now also R39.2, U3.4 (I4); no longer R29.2
- net A_Enable_HV: now also D11.1 (K), J40.9 (Pin_9), U3.13 (O4); no longer D10.1 (K)
- net A_Step: now also R38.2, U3.5 (I5); no longer R30.2
- net A_Step_HV: now also D12.1 (K), J40.11 (Pin_11), U3.12 (O5); no longer D11.1 (K)
- net B_Dir: now also R47.2, U3.3 (I3); no longer R34.2
- net B_Dir_HV: now also D17.1 (K), J5.13 (Pin_13), U3.14 (O3); no longer D15.1 (K)
- net B_Enable: now also R49.2, U3.1 (I1); no longer R32.2
- net B_Enable_HV: now also D15.1 (K), J5.9 (Pin_9), U3.16 (O1); no longer D13.1 (K)
- net B_Step: now also R48.2, U3.2 (I2); no longer R33.2
- net B_Step_HV: now also D16.1 (K), J5.11 (Pin_11), U3.15 (O2); no longer D14.1 (K)
- net C_Dir: now also R44.2, U3.6 (I6); no longer R37.2
- net C_Dir_HV: now also D32.1 (K), J8.13 (Pin_13), U3.11 (O6); no longer D18.1 (K)
- net C_Enable: now also R46.2, U3.4 (I4); no longer R35.2
- net C_Enable_HV: now also D18.1 (K), J8.9 (Pin_9), U3.13 (O4); no longer D16.1 (K)
- net C_Step: now also R45.2, U3.5 (I5); no longer R36.2
- net C_Step_HV: now also D31.1 (K), J8.11 (Pin_11), U3.12 (O5); no longer D17.1 (K)
- net I2S_BCK: no longer U5.36 (GPIO22)
- net I2S_DATA: now also U5.36 (GPIO22); no longer U5.33 (GPIO21)
- net I2S_WS: now also U5.33 (GPIO21); no longer U5.28 (GPIO17)
- net SCL: now also J31.3 (Pin_3), J42.3 (Pin_3), J47.3 (Pin_3), J52.3 (Pin_3)
- net SDA: now also J32.3 (Pin_3), J41.3 (Pin_3), J46.3 (Pin_3), J51.3 (Pin_3)
- net X_Dir: now also R33.2, U3.3 (I3); no longer R3.2
- net X_Dir_HV: now also J40.5 (Pin_5), U3.14 (O3)
- net X_Enable: now also R35.2, U3.1 (I1); no longer R1.2
- net X_Enable_HV: now also J40.1 (Pin_1), U3.16 (O1)
- net X_Step: now also R34.2, U3.2 (I2); no longer R2.2
- net X_Step_HV: now also J40.3 (Pin_3), U3.15 (O2)
- net Y_Dir: now also R30.2, U3.6 (I6); no longer R6.2
- net Y_Dir_HV: now also J5.5 (Pin_5), U3.11 (O6)
- net Y_Enable: now also R32.2, U3.4 (I4)
- net Y_Enable_HV: now also J5.1 (Pin_1), U3.13 (O4)
- net Y_Step: now also R31.2, U3.5 (I5); no longer R5.2
- net Y_Step_HV: now also J5.3 (Pin_3), U3.12 (O5)
- net Z_Dir: now also R40.2, U12.11 (I0c), U2.1 (Q1), U3.3 (I3); no longer R9.2
- net Z_Dir_HV: now also D10.1 (K), J8.5 (Pin_5), U3.14 (O3); no longer D9.1 (K)
- net Z_Enable: now also R42.2, U3.1 (I1); no longer R7.2
- net Z_Enable_HV: now also D8.1 (K), J8.1 (Pin_1), U3.16 (O1); no longer D7.1 (K)
- net Z_Step: now also R41.2, U12.5 (I0b), U2.2 (Q2), U3.2 (I2); no longer R8.2
- net Z_Step_HV: now also D9.1 (K), J8.3 (Pin_3), U3.15 (O2); no longer D8.1 (K)
- net at R2.1: now also D3.2 (A); no longer R20.2
- net at R1.1: now also D2.2 (A); no longer R19.2
- net at D13.2 (A): now also R13.1; no longer R41.1
- net at R3.1: now also D4.2 (A); no longer R21.2
- net at R26.2: now also D19.1 (K), D21.2 (L1); no longer R8.1
- net at R18.1: now also D18.2 (A); no longer D9.2 (A)
- net at R69.2: now also J40.14 (Pin_14)
- net at R59.2: now also J8.10 (Pin_10)
- net at R60.2: now also J8.12 (Pin_12)
- net at R61.2: now also J8.14 (Pin_14)
- net at R11.1: now also D11.2 (A); no longer D2.2 (A)
- net at D10.2 (A): now also R9.1; no longer R38.1
- net at R27.2: now also R26.1, U9.8 (VBUS); no longer R9.1
- net at U16.10 (7): now also J41.2 (Pin_2)
- net at U16.11 (8): now also J42.2 (Pin_2)
- net at U13.10 (7): now also J32.2 (Pin_2)
- net at U13.11 (8): now also J31.2 (Pin_2)
- net at U13.8 (5): now also J35.2 (Pin_2)
- net at U13.9 (6): now also J34.2 (Pin_2)
- net at D16.2 (A): now also R16.1; no longer R44.1
- net at R58.2: now also J40.6 (Pin_6)
- net at R54.2: now also R25.1, R53.2, U29.6 (A); no longer R36.1
- net at R65.2: now also J5.14 (Pin_14)
- net at R62.2: now also J8.16 (Pin_16)
- net at R63.2: now also J5.10 (Pin_10)
- net at R64.2: now also J5.12 (Pin_12)
- net at R5.1: now also D6.2 (A); no longer R23.2
- net at R68.2: now also J40.12 (Pin_12)
- net at R70.2: now also J40.16 (Pin_16)
- net at U22.11 (8): now also J52.2 (Pin_2)
- net at R7.1: now also D8.2 (A); no longer R25.2
- net at R66.2: now also J5.16 (Pin_16)
- net at R82.1: now also R73.2, U30.2 (-)
- net at R57.2: now also J40.4 (Pin_4)
- net at R14.1: now also D14.2 (A); no longer D5.2 (A)
- net at R6.1: now also D7.2 (A)
- net EXT_Z_Enable: now reaches U12.3 (I1a)
- net at D12.2 (A): now also R12.1; no longer R40.1
- net at U19.10 (7): now also J46.2 (Pin_2)
- net at R67.2: now also J40.10 (Pin_10)
- net at U19.11 (8): now also J47.2 (Pin_2)
- net at D17.2 (A): now also R17.1; no longer R45.1
- net at R56.2: now also J40.2 (Pin_2)
- net at U22.10 (7): now also J51.2 (Pin_2)
- net at D15.2 (A): now also R15.1; no longer R43.1
- net PWM1: now reaches R86.1
- net PWM1: now also R114.2
- net A_CC1 renamed CC1
- net A_CC2 renamed CC2
- net A_CS_SD renamed CS_SD
- net CS_SD: now also U23.6 (SD0/DO)
- net A_D+ renamed D+
- net A_D- renamed D-
- net A_DTR renamed DTR
- net A_GPIO_0 renamed GPI_0
- net GPI_0: now also C24.1, R22.1, R120.2, SW12.2, U24.16
- net A_GPIO_1 renamed TXD0
- net TXD0: now also U9.20 (RXD)
- net A_GPIO_16 renamed RS485_RX
- net RS485_RX: now also R71.1, D35.1 (K), U29.1 (RO)
- net A_GPIO_25 renamed A_LIM
- net A_LIM: now also R128.2, U26.16
- net A_GPIO_26 renamed B_LIM
- net B_LIM: now also R129.2, U26.14
- net A_GPIO_27 renamed C_LIM
- net C_LIM: now also R130.2, U26.12
- net A_GPIO_3 renamed RXD0
- net RXD0: now also U9.21 (TXD)
- net A_GPIO_32 renamed Y_LIM
- net Y_LIM: now also R126.2, U25.12
- net A_GPIO_33 renamed Z_LIM
- net A_GPIO_36 renamed MACRO_1
- net MACRO_1: now also R122.2, U24.12
- net A_GPIO_39 renamed MACRO_2
- net MACRO_2: now also R123.2, U24.10
- net A_GPIO_4 renamed PWM2
- net PWM2: now also R115.2, R116.1
- net A_GPIO_5 renamed RS485_EN
- net RS485_EN: now also R72.1, U29.2 (~{RE}), U29.3 (DE)
- net A_MISO renamed MISO
- net MISO: now also J31.1 (Pin_1), J42.1 (Pin_1), J47.1 (Pin_1), J52.1 (Pin_1)
- removed net A_MOSI: J16.3 (CMD), U16.9 (6), U19.9 (6), U22.9 (6), U5.16 (MTCK/GPIO13/ADC2_CH4)
- net A_RESET renamed RESET
- net RESET: now also C25.1, R121.2, U24.14; no longer C1.2
- net A_RTS renamed RTS
- net A_RXD0 renamed MACRO_3
- net MACRO_3: now also R124.2, U25.16; no longer U9.21 (TXD)
- removed net A_SCLK: J16.5 (CLK), U16.8 (5), U19.8 (5), U22.8 (5), U5.13 (MTMS/GPIO14/ADC2_CH6)
- net A_TXD0 renamed X_LIM
- net X_LIM: now also R125.2, U25.14; no longer U9.20 (RXD)
- removed net B_VCC: C24.1, C25.1, C26.1, R86.2, U12.16 (VCC)
- net I2S0_11 renamed RLY_3
- net RLY_3: now also R43.2, U3.7 (I7)
- net I2S0_14 renamed RLY_2
- net RLY_2: now also R36.2, U3.7 (I7)
- net I2S0_3 renamed RLY_1
- net RLY_1: now also R29.2, U3.7 (I7)
- net MUX_SET renamed EXT_MUX_EN
- net EXT_MUX_EN: now also R119.2
- removed net Z_Dir_GRBL: U12.5 (I0b), U2.1 (Q1)
- net Z_Dir_THC renamed EXT_Z_Step
- removed net Z_Step_GRBL: U12.11 (I0c), U2.2 (Q2)
- net Z_Step_THC renamed EXT_Z_Dir
- new net: D3.2 (A), R30.1, R38.2
- new net: J12.1 (Pin_1), R30.2
- new net: J5.2 (Pin_2), R106.2
- new net: J5.4 (Pin_4), R107.2
- new net: J5.6 (Pin_6), R108.2
- new net: J5.8 (Pin_8), R109.2
- new net: C7.1, D3.1 (K), FB2.1, R35.1, R36.1, R37.1, U2.1 (IN), U2.3 (EN), U3.8 (VDD)
- new net: J8.2 (Pin_2), R110.2
- new net: J8.4 (Pin_4), R111.2
- new net: J8.6 (Pin_6), R112.2
- new net: J8.8 (Pin_8), R113.2
- new net: D36.1 (K), D39.1 (K), J24.4 (Pin_4), R23.1
- new net: D37.1 (K), D39.2 (A), J24.5 (Pin_5), R54.1
- new net: R4.2, U25.5
- new net: J28.5 (Pin_5), U25.6
- new net: J44.2 (Pin_2), U19.8 (5)
- new net: R4.2, U26.3
- new net: J29.2 (Pin_2), U26.4
- new net: R4.2, U24.7
- new net: J26.2 (Pin_2), U24.8
- new net: C1.1, R86.2, U30.3 (+)
- new net: J36.2 (Pin_2), U16.3 (VCC)
- new net: J37.2 (Pin_2), U16.8 (5)
- new net: J38.2 (Pin_2), U16.9 (6)
- new net: J25.2 (Pin_2), U13.3 (VCC)
- new net: D34.2 (A), R50.1
- new net: J50.2 (Pin_2), U22.9 (6)
- new net: J6.2 (Pin_2), R59.1, R60.1, R61.1, R62.1
- new net: J3.2 (Pin_2), R110.1, R111.1, R112.1, R113.1
- new net: J4.2 (Pin_2), R105.1, R56.1, R57.1, R58.1
- new net: R23.2, R25.2, R52.1, U29.7 (B)
- new net: J12.2 (Pin_2), R31.1
- new net: R117.1, R118.2, U30.6 (-)
- new net: D2.1 (K), R31.2, R39.2
- new net: C6.2, C7.2, D2.2 (A), FB1.2, R34.2, U2.2 (GND), U3.3 (GND)
- new net: R131.2, U26.10
- new net: D33.2 (A), R21.1
- new net: R4.2, U26.7
- new net: R4.2, U24.1
- new net: R73.1, RV1.1
- new net: R4.2, U26.5
- new net: D5.2 (A), R4.1
- new net: J48.2 (Pin_2), U22.3 (VCC)
- new net: D9.2 (A), R8.1
- new net: R118.1, RV2.1
- new net: J2.2 (Pin_2), R106.1, R107.1, R108.1, R109.1
- new net: J30.5 (Pin_5), U26.6
- new net: D35.2 (A), R51.1
- new net: R34.1, U3.1 (ADDR)
- new net: J15.11 (Pin_11), R36.2, U3.10 (SCL)
- new net: J15.9 (Pin_9), R37.2, U3.2 (ALERT/RDY)
- new net: C3.1, R32.2, R38.1, U3.4 (AIN0)
- new net: C3.2, R33.1, R39.1, U3.5 (AIN1)
- new net: J15.10 (Pin_10), R35.2, U3.9 (SDA)
- new net: R127.2, U25.10
- new net: C40.1, R116.2, U30.5 (+)
- new net: C8.2, FB1.1, J15.1 (Pin_1), J15.12 (Pin_12)
- new net: C8.1, FB2.2, J15.3 (Pin_3)
- new net: J29.5 (Pin_5), U26.2
- new net: J33.2 (Pin_2), R67.1, R68.1, R69.1, R70.1
- new net: R4.2, U24.3
- new net: J7.2 (Pin_2), R63.1, R64.1, R65.1, R66.1
- new net: J30.2 (Pin_2), U26.8
- new net: D31.2 (A), R19.1
- new net: C6.1, R32.1, R33.2, U2.5 (OUT)
- new net: R4.2, U25.3
- new net: J43.2 (Pin_2), U19.3 (VCC)
- new net: J45.2 (Pin_2), U19.9 (6)
- new net: J40.8 (Pin_8), R105.2
- new net: J39.5 (Pin_5), U24.2
- new net: R4.2, U25.1
- new net: J27.5 (Pin_5), U25.2
- new net: J39.2 (Pin_2), U24.4
- new net: R4.2, U24.5
- new net: D32.2 (A), R20.1
- new net: J49.2 (Pin_2), U22.8 (5)
- new net: J26.5 (Pin_5), U24.6
- new net: R4.2, U26.1
- new net: R4.2, U25.7
- new net: J28.2 (Pin_2), U25.8
- new net: J27.2 (Pin_2), U25.4
- new net I2S0_11_HV: D33.1 (K)
- new net MOSI: J16.3 (CMD), J34.3 (Pin_3), J38.3 (Pin_3), J45.3 (Pin_3), J50.3 (Pin_3), U23.5 (CMD/DI), U5.16 (MTCK/GPIO13/ADC2_CH4)
- new net PWM1_10V: RV1.2, U30.1
- new net PWM2_10V: RV2.2, U30.7
- new net RLY_1_HV: D30.1 (K), D7.1 (K), K2.A1, U3.10 (O7)
- new net RLY_2_HV: D14.1 (K), D26.1 (K), K1.A1, U3.10 (O7)
- new net RLY_3_HV: D38.1 (K), K3.A1, U3.10 (O7)
- new net RS485_TX: D34.1 (K), R55.1, U29.4 (DI), U5.28 (GPIO17)
- new net SCLK: J16.5 (CLK), J35.3 (Pin_3), J37.3 (Pin_3), J44.3 (Pin_3), J49.3 (Pin_3), U23.3 (CLK), U5.13 (MTMS/GPIO14/ADC2_CH6)
- no-connect marks 98 -> 96
Other:
- note added: "0-10V Analog Output"
- note added: "1 -- GND 2 -- +12V 3 -- +5V or + 3V3 4 -- GPIO OR DAC 5 -- GPIO OR PWM 6 -- GPIO OR ADC+ 7 -- GPIO OR ADC- 8 -- SPI_SCLK OR GPIO 9 -- SPI_MOSI OR GPIO 10 - SPI_CS OR I2C_SDA 11 - SPI_MISO OR I2C_SCL 12 - GND"
- note added: "1.5V"
- note added: "Jumper to module #3"
- note added: "Opto Inputs"
- note added: "RS485"
- note added: "Relay Outputs"
- note added: "Shift Register & Stepper Outputs"
- note added: "USB to Serial"
- note added: "extra 5v outputs"
- note removed: "CoProcessor ESP32"
- note removed: "Expansion Modules For CoProcessor"
- note removed: "Stepper Outputs & Level Shifting"
- note removed: "uart???"
- moved on the sheet: C10, C11, C12, C13, C14, C15, C16, C17, C18, C19, C2, C20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

Commit message: start a teensy version with migration to grblHAL for built in THC
Parts:
- removed C26, C38: 100nF, Capacitor_SMD:C_0603_1608Metric, symbol Device:C_Small
- removed C34: 22uF, Capacitor_SMD:C_1206_3216Metric, symbol Device:C_Small
- removed C35: 10uF, Capacitor_SMD:C_0805_2012Metric, symbol Device:C_Small
- removed C36: 4.7uF, Capacitor_SMD:C_0805_2012Metric, symbol Device:C_Small
- removed C37: 1uF, Capacitor_SMD:C_0805_2012Metric, symbol Device:C_Small
- removed C39: 10nF, Capacitor_SMD:C_0603_1608Metric, symbol Device:C_Small
- removed D26, D30, D38: D_Small, symbol Device:D_Small
- removed D29: D_Schottky, symbol Device:D_Schottky
- removed K3: G2RL-1-E-DC12, Relay_THT:Relay_SPDT_Schrack-RT1-16A-FormC_RM5mm, symbol Relay:RT314A12
- removed R105, R109, R113, R62, R66, R70: 510R, Resistor_SMD:R_0603_1608Metric, symbol Device:R_Small
- removed R119: 10K, Resistor_SMD:R_0603_1608Metric, symbol Device:R_Small
- removed R4 (x12): 2K, Resistor_SMD:R_0603_1608Metric_Pad0.98x0.95mm_HandSolder, symbol Device:R_Small
- removed R76: 100K, Resistor_SMD:R_0603_1608Metric, symbol Device:R_Small
- removed U12: 74LVC157A, Package_SO:SOP-16_3.9x9.9mm_P1.27mm, symbol 111_Torban_Symbols:74LVC157A
- removed U4: 74AHCT595PW, Package_SO:TSSOP-16-1EP_4.4x5mm_P0.65mm, symbol 111_Torban_Symbols:74AHC595
- removed U8: AP2112K-3.3, Package_TO_SOT_SMD:SOT-23-5, symbol Regulator_Linear:AP2112K-3.3
- added C10, C11, C14, C15, C16, C17, C18, C19, C2, C20, C21, C4, C40, C5, C6, C8, C9: 100nF, Capacitor_SMD:C_0603_1608Metric, symbol Device:C_Small
- added D1, D10, D11, D12, D13, D14, D15, D16, D2, D3, D4, D5, D6, D7, D8, D9: Emerald, LED_SMD:LED_0603_1608Metric, symbol Device:LED_Small_Filled
- added D3 (x2): SS510, Diode_SMD:D_SMC, symbol PCM_Diode_Schottky_AKL:SS510
- added J11, J8, J9: Conn_02x03_Top_Bottom, KiCad:DB2ERH-2.5-2-3P-GN, symbol Connector_Generic:Conn_02x03_Top_Bottom
- added JP1, JP2, JP3: A0, symbol Jumper:SolderJumper_2_Bridged
- added Q1 (x3): BSS138, Package_TO_SOT_SMD:SOT-23, symbol Transistor_FET:BSS138
- added R10, R11, R12, R13, R14, R15, R27, R28, R29, R30, R31, R32, R33, R34, R36, R37, R38, R39, R40, R41, R42, R52, R53, R54, R55, R56, R57, R58, R59, R8, R9: 1K, Resistor_SMD:R_0603_1608Metric, symbol Device:R_Small
- added R16, R19 (x3), R26, R35, R45 (x3), R48, R49, R50, R51, R90, R91: 10K, Resistor_SMD:R_0603_1608Metric, symbol Device:R_Small
- added U4: PCA9555PW, Package_SO:TSSOP-24_4.4x7.8mm_P0.65mm, symbol Interface_Expansion:PCA9555PW
- added U6: ESP32_38p, KiCad:MH ET LIVE ESP-32 Dev Kit, symbol 111_Torban_Symbols:MH-ET-LIVE-ESP32
- added U8: ELQ3H7, KiCad:ELQ3H7 SOP-16_4.4x10.4mm_P1.27mm, symbol Isolator:LTV-847S
- added U9: AZ1117EH-3.3TRG1, Package_TO_SOT_SMD:SOT-223-3_TabPin2, symbol Regulator_Linear:AMS1117-3.3
- R113: renamed from R10; LCSC C21190 -> (none)
- R114: renamed from R1; LCSC C21190 -> (none)
- R115: renamed from R2; LCSC C21190 -> (none)
- R116: renamed from R3; LCSC C21190 -> (none)
- R117: renamed from R4; LCSC C21190 -> (none)
- R118: renamed from R5; LCSC C21190 -> (none)
- R119: renamed from R6; LCSC C21190 -> (none)
- R129: renamed from R7; LCSC C21190 -> (none)
- R130: renamed from R8; LCSC C21190 -> (none)
- R131: renamed from R9; LCSC C21190 -> (none)
- R132: renamed from R11; LCSC C21190 -> (none)
- R133: renamed from R12; LCSC C21190 -> (none)
- R134: renamed from R13; LCSC C21190 -> (none)
- R135: renamed from R14; LCSC C21190 -> (none)
- R145: renamed from R15; LCSC C21190 -> (none)
- R146: renamed from R16; LCSC C21190 -> (none)
- R147: renamed from R17; LCSC C21190 -> (none)
- R148: renamed from R18; LCSC C21190 -> (none)
- R149: renamed from R19; LCSC C21190 -> (none)
- R150: renamed from R20; LCSC C21190 -> (none)
- R151: renamed from R21; LCSC C21190 -> (none)
- R30, R32, R33: footprint Resistor_SMD:R_0603_1608Metric_Pad0.98x0.95mm_HandSolder -> Resistor_SMD:R_0603_1608Metric; LCSC C22548 -> (none)
- R43: value 10K -> 1K; LCSC C25804 -> (none)
- R71: renamed from R50; LCSC C21190 -> (none)
- R73: renamed from R51; LCSC C21190 -> (none)
- R74: renamed from R73; LCSC C21190 -> (none)
- R75: renamed from R118; LCSC C21190 -> (none)
- R83: renamed from R23; LCSC C21190 -> (none)
- R84: renamed from R54; LCSC C21190 -> (none)
- R88: renamed from R79; LCSC C21190 -> (none)
- renumbered C24 to C1, C2 to C12, C3 to C13, C12 to C22, C14 to C23, C17 to C24, C8 to C25, C1 to C26, C40 to C27, C21 to C28, C16 to C29, C25 to C3, C23 to C30, C22 to C31, C19 to C32, C20 to C33, C10 to C34, C9 to C35, C15 to C36, C11 to C37, C18 to C38, C13 to C39, C4 to C41, C5 to C42, C6 to C43, D34 to D20, D35 to D22, D20 to D25, D25 to D26, D36 to D27, D39 to D28, D37 to D29, D23 to D30, D22 to D31, D1 to D32, D2 to D33, D3 to D34, D4 to D35, D5 to D36, D6 to D37, D7 to D38, D8 to D39, D9 to D40, D10 to D41, D11 to D42, D12 to D43, D13 to D44, D14 to D45, D15 to D46, D16 to D47, D17 to D48, D18 to D49, D31 to D50, D32 to D51, D33 to D52, J29 to J1, J24 to J10, J25 to J13, J43 to J14, J35 to J15, J34 to J16, J32 to J17, J31 to J18, J44 to J19, J30 to J2, J45 to J20, J46 to J21, J47 to J22, J36 to J23, J48 to J24, J33 to J25, J7 to J26, J6 to J27, J37 to J28, J38 to J29, J27 to J3, J41 to J30, J42 to J31, J49 to J32, J50 to J33, J51 to J34, J52 to J35, J40 to J36, J5 to J37, J8 to J38, J4 to J39, J28 to J4, J2 to J40, J3 to J41, J9 to J42, J10 to J43, J12 to J45, J13 to J46, J14 to J47, J15 to J48, J16 to J49, J17 to J50, J18 to J51, J19 to J53, J20 to J54, J21 to J55, J22 to J56, J23 to J57, J39 to J6, J26 to J7, JP1 to JP4, JP2 to JP5, K2 to K1, K1 to K3, L3 to L1, L1 to L2, L2 to L3, Q19 to Q4, Q20 to Q5, R45 to R100, R32 to R101, R39 to R102, R46 to R103, R33 to R104, R40 to R105, R47 to R106, R34 to R107, R41 to R108, R48 to R109, R35 to R110, R42 to R111, R49 to R112, R67 to R120, R68 to R121, R69 to R122, R63 to R123, R64 to R124, R65 to R125, R59 to R126, R60 to R127, R61 to R128, R56 to R136, R57 to R137, R58 to R138, R106 to R139, R107 to R140, R108 to R141, R110 to R142, R111 to R143, R112 to R144, R128 to R17, R129 to R18, R130 to R19, R131 to R20, R124 to R21, R125 to R22, R126 to R23, R127 to R24, R28 to R25, R22 to R4, R120 to R44, R121 to R45, R122 to R46, R123 to R47, R74 to R60, R75 to R61, R72 to R62, R114 to R63, R115 to R64, R86 to R65, R116 to R66, R71 to R67, R55 to R68, R82 to R69, R117 to R70, R26 to R72, R27 to R76, R83 to R78, R84 to R79, R52 to R80, R25 to R81, R53 to R82, R80 to R86, R81 to R87, R78 to R89, R29 to R92, R36 to R93, R30 to R95, R37 to R96, R44 to R97, R31 to R98, R38 to R99, SW12 to SW1, SW1 to SW2, U23 to U1, U30 to U10, U10 to U11, U7 to U12, U29 to U13, U9 to U14, U1 to U16, U2 to U17, U3 to U18, U13 to U19, U26 to U2, U19 to U20, U16 to U24, U22 to U25, U25 to U3, U24 to U7, U6 to U9
Connections:
- net I2S0_11_HV is gone; now on net RLY_3_HV: D52.1 (K)
- net +12V: now also J36.16 (Pin_16), J36.8 (Pin_8), J37.16 (Pin_16), J37.8 (Pin_8), J38.16 (Pin_16), J38.8 (Pin_8), R17.1, R18.1, R19.1, R20.1, R21.1, R22.1, R23.1, R24.1, R43.2, R44.1, R45.1, R46.1, R47.1, C10.2, C11.2, C14.2, C15.2, C16.2, C17.2, C18.2, C19.2, C2.1, C2.2, C20.2, C21.2, C4.2, C40.1, C40.2, C5.2, C6.2, C8.2, C9.2, D3.2 (A), D3.2 (A), J8.1 (Pin_1), J8.3 (Pin_3), J8.4 (Pin_4), J8.6 (Pin_6), J9.1 (Pin_1), J9.3 (Pin_3), J9.4 (Pin_4), J9.6 (Pin_6), JP1.1 (A), JP2.1 (A), JP3.1 (A), R10.2, R11.2, R12.2, R13.2, R14.2, R15.2, R16.2, R19.2, R19.2, R19.2, R26.2, R35.2, R36.2, R37.2, R38.2, R39.2, R40.2, R41.2, R42.2, R48.1, R49.1, R50.1, R51.1, R8.2, R9.2, R90.2, R91.1, R91.2, U4.12 (VSS), U4.24 (VDD), U6.13 (GND), U6.19 (GND), U6.33 (GND), U6.38 (VIN), U8.11, U8.13, U8.15, U8.9, U9.1 (GND), U9.3 (VI); no longer C7.1, R43.1
- net +3V3: now also Q1.1 (G), Q1.1 (G), Q1.1 (G), R45.2, R45.2, R45.2, U6.20 (3.3V), U9.2 (VO); no longer R17.1, R18.1, R19.1, R20.1, R21.1, R22.1, R23.1, R24.1, R44.1, R45.1, R46.1, R47.1
- net CS_SD: now also U6.4 (IO15)
- net GPI_0: now also U6.6 (IO0); no longer C1.1, R4.1, R44.2, SW1.2, U5.25 (GPIO0/BOOT/ADC2_CH1), U7.16
- net I2S_BCK: now also R90.1, U6.18 (IO23)
- net I2S_DATA: now also U6.17 (IO22)
- net I2S_WS: now also U6.14 (IO21)
- net MACRO_1: now also C19.1, R57.1, U4.17 (IO1_4); no longer R46.2, U5.4 (SENSOR_VP/GPIO36/ADC1_CH0), U7.12
- net MACRO_2: now also C18.1, R56.1, U4.18 (IO1_5); no longer R47.2, U5.5 (SENSOR_VN/GPIO39/ADC1_CH3), U7.10
- net MACRO_3: now also C21.1, R59.1, U4.19 (IO1_6); no longer R21.2, U3.16, U5.6 (GPIO34/ADC1_CH6)
- net MISO: now also U6.32 (IO12)
- net MOSI: now also U6.34 (IO13)
- net PWM1: now also U6.5 (IO2)
- net PWM1_10V: now also J10.1 (Pin_1)
- net PWM2: now also U6.7 (IO4)
- net PWM2_10V: now also J10.2 (Pin_2)
- net RESET: now also U6.21 (RST); no longer R45.2, U7.14
- net RLY_1_HV: now also D3.1 (K)
- net RLY_2: now also U17.3 (Q3); no longer U17.6 (Q6)
- net RLY_2_HV: now also D3.1 (K)
- net RLY_3_HV: no longer U3.10 (O7)
- net RS485_EN: now also U6.10 (IO5)
- net RS485_RX: now also U6.8 (IO16)
- net RS485_TX: now also U6.9 (IO17)
- net RXD0: now also U6.15 (RXD)
- net SCL: now also Q1.2 (S), R45.1, U6.12 (IO19)
- net SCLK: now also U6.31 (IO14)
- net SDA: now also Q1.2 (S), R45.1, U6.11 (IO18)
- net TXD0: now also U6.16 (TXD)
- net B_DEBUG: now reaches J37.15 (Pin_15)
- net B_DEBUG: now also C10.1, R33.1, U4.11 (IO0_7)
- net Y_DEBUG: now reaches J37.7 (Pin_7)
- net Y_DEBUG: now also C8.1, R31.1, U4.9 (IO0_5)
- net C_DEBUG: now reaches J38.15 (Pin_15)
- net C_DEBUG: now also C16.1, R54.1, U4.16 (IO1_3)
- net Z_DEBUG: now reaches J38.7 (Pin_7)
- net Z_DEBUG: now also C14.1, R52.1, U4.14 (IO1_1)
- net at U3.5: now also R14.1
- net at U3.6: now also D7.2 (A); no longer J4.5 (Pin_5)
- net at U2.3: now also R9.1
- net at U2.4: now also D2.2 (A); no longer J1.2 (Pin_2)
- net at U7.7: now also R39.1
- net at U7.8: now also D12.2 (A); no longer J7.2 (Pin_2)
- net Q7S_1: now reaches U16.9 (Q7S), U17.14 (DS)
- net Q7S_2: now reaches U17.9 (Q7S), U18.14 (DS)
- net at R20.2, U2.10: now also R30.2
- net at U2.7: now also R11.1
- net at U7.1: now also R36.1
- net at U2.5: now also R10.1
- net at U2.6: now also D3.2 (A); no longer J2.5 (Pin_5)
- net at R24.2, U3.10: now also R34.2
- net at J1.5 (Pin_5): now also D1.1 (K); no longer U2.2
- net at U7.3: now also R37.1
- net RLY_1_COM: now reaches K1.11
- net RLY_1_COM: now also J11.2 (Pin_2)
- net RLY_1_NC: now reaches K1.12
- net RLY_1_NC: now also J11.3 (Pin_3)
- net RLY_1_NO: now reaches K1.14
- net RLY_1_NO: now also J11.1 (Pin_1)
- net at J2.2 (Pin_2): now also D4.1 (K); no longer U2.8
- net at U3.3: now also R13.1
- net A_DEBUG: now reaches J36.15 (Pin_15)
- net A_DEBUG: now also C6.1, R29.1, U4.7 (IO0_3)
- net X_DEBUG: now reaches J36.7 (Pin_7)
- net X_DEBUG: now also C4.1, R27.1, U4.5 (IO0_1)
- net at U7.2: now also D9.2 (A); no longer J6.5 (Pin_5)
- net at U3.1: now also R12.1
- net at U3.2: now also D5.2 (A); no longer J3.5 (Pin_5)
- net at J6.2 (Pin_2): now also D10.1 (K); no longer U7.4
- net at U7.5: now also R38.1
- net RLY_2_COM: now reaches K3.11
- net RLY_2_COM: now also J11.5 (Pin_5)
- net RLY_2_NC: now reaches K3.12
- net RLY_2_NC: now also J11.6 (Pin_6)
- net RLY_2_NO: now reaches K3.14
- net RLY_2_NO: now also J11.4 (Pin_4)
- net at U7.6: now also D11.2 (A); no longer J7.5 (Pin_5)
- net at U2.1: now also R8.1
- net at U3.7: now also R15.1
- net at J4.2 (Pin_2): now also D8.1 (K); no longer U3.8
- net at J3.2 (Pin_2): now also D6.1 (K); no longer U3.4
- net A_LIM: no longer names the net of R17.2, U2.16
- net A_LIM: now also R27.2; no longer U5.10 (DAC_1/ADC2_CH8/GPIO25)
- net B_LIM: no longer names the net of R18.2, U2.14
- net B_LIM: now also R28.2; no longer U5.11 (DAC_2/ADC2_CH9/GPIO26)
- net C_LIM: no longer names the net of R19.2, U2.12
- net C_LIM: now also R29.2; no longer U5.12 (ADC2_CH7/GPIO27)
- removed net RLY_3: R43.2, U17.3 (Q3), U3.7 (I7)
- net X_LIM: no longer names the net of R22.2, U3.14
- net X_LIM: now also R32.2; no longer U5.7 (GPIO35/ADC1_CH7)
- net Y_LIM: no longer names the net of R23.2, U3.12
- net Y_LIM: now also R33.2; no longer U5.8 (32K_XP/GPIO32/ADC1_CH4)
- net Z_LIM renamed IO33
- net IO33: now also U6.27 (IO33)
- new net: R50.2, R58.2, U8.12
- new net: R42.1, U8.5
- new net: D15.2 (A), U8.6
- new net: JP3.2 (B), R35.1, U4.21 (A0)
- new net: R47.2, R55.2, U7.10
- new net: D10.2 (A), U7.4
- new net: D14.1 (K), J8.2 (Pin_2)
- new net: D13.1 (K), J8.5 (Pin_5)
- new net: R44.2, R52.2, U7.16
- new net: JP2.2 (B), R26.1, U4.2 (A1)
- new net: D16.1 (K), J9.2 (Pin_2)
- new net: D16.2 (A), U8.8
- new net: R51.2, R59.2, U8.10
- new net: R46.2, R54.2, U7.12
- new net: R40.1, U8.1
- new net: R43.1, U8.7
- new net: D2.1 (K), J1.2 (Pin_2)
- new net: D6.2 (A), U3.4
- new net: D1.2 (A), U2.2
- new net: R48.2, R56.2, U8.16
- new net: D13.2 (A), U8.2
- new net: R21.2, R31.2, U3.16
- new net: R45.2, R53.2, U7.14
- new net: D8.2 (A), U3.8
- new net: D3.1 (K), J2.5 (Pin_5)
- new net: JP1.2 (B), R16.1, U4.3 (A2)
- new net: D12.1 (K), J7.2 (Pin_2)
- new net: R49.2, R57.2, U8.14
- new net: R41.1, U8.3
- new net: D14.2 (A), U8.4
- new net: D9.1 (K), J6.5 (Pin_5)
- new net: D15.1 (K), J9.5 (Pin_5)
- new net: D5.1 (K), J3.5 (Pin_5)
- new net: D7.1 (K), J4.5 (Pin_5)
- new net: D4.2 (A), U2.8
- new net: D11.1 (K), J7.5 (Pin_5)
- new net A_LIM+: C7.1, R30.1, U4.6 (IO0_2)
- new net B_LIM+: C11.1, R34.1, U4.10 (IO0_6)
- new net C_LIM+: C17.1, R55.1, U4.15 (IO1_2)
- new net EXIO_INT: Q1.2 (S), R45.1, U5.5 (SENSOR_VN/GPIO39/ADC1_CH3), U6.23 (IO39)
- new net EXIO_INT_5: Q1.3 (D), R19.1, U4.1 (~{INT})
- new net I2S0_14: U17.6 (Q6)
- new net IO0: C1.1, R4.1, SW1.2, U5.25 (GPIO0/BOOT/ADC2_CH1)
- new net IO25: U5.10 (DAC_1/ADC2_CH8/GPIO25), U6.28 (IO25)
- new net IO26: U5.11 (DAC_2/ADC2_CH9/GPIO26), U6.29 (IO26)
- new net IO27: U5.12 (ADC2_CH7/GPIO27), U6.30 (IO27)
- new net IO32: U5.8 (32K_XP/GPIO32/ADC1_CH4), U6.26 (IO32)
- new net IO34: U5.6 (GPIO34/ADC1_CH6), U6.24 (IO34)
- new net IO35: U5.7 (GPIO35/ADC1_CH7), U6.25 (IO35)
- new net IO36: U5.4 (SENSOR_VP/GPIO36/ADC1_CH0), U6.22 (IO36)
- new net MACRO_4: C20.1, R58.1, U4.20 (IO1_7)
- new net SCL_5V: Q1.3 (D), R19.1, U4.22 (SCL)
- new net SDA_5V: Q1.3 (D), R19.1, U4.23 (SDA)
- new net X_LIM+: C5.1, R28.1, U4.4 (IO0_0)
- new net Y_LIM+: C9.1, R32.1, U4.8 (IO0_4)
- new net Z_LIM+: C15.1, R53.1, U4.13 (IO1_0)
- no-connect marks 96 -> 103
Other:
- note added: "24V -> 5V@3A Buck Supply & 3V3 LDO"
- note added: "LED 3.3V Vf OPTO 1.4V Vf"
- note added: "OK-2023-09-23"
- note added: "Opto Inputs x16"
- note removed: "24V -> 5V@3A Buck Supply"
- note removed: "3V3 ESP32 Voltage Regulators"
- note removed: "Opto Inputs"
- note removed: "Z-Interceptor"
- moved on the sheet: C1, C12, C13, C22, C23, C24, C26, C27, C28, C3, C30, C34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
