File: Hardware/Input Module/4 Channel Screw term/4 Channel Screw term.kicad_sch (KiCad schematic)
At the start: 22 parts, among them J1 Screw_Terminal_01x06, J2 Screw_Terminal_01x06, J5 Conn_01x12_Male, U1 LTV-847S, U2 74HC7014

Commit message: redesigned input and output modules, cleaned some files, ordered 10 of each
Parts:
- U1: footprint Package_SO:SOP-16_4.4x10.4mm_P1.27mm -> Package_DIP:SMDIP-16_W9.53mm
- U2: footprint Package_SO:TSSOP-14_4.4x5mm_P0.65mm -> Package_SO:SO-14_3.9x8.65mm_P1.27mm
Other:
- company: (none) -> Torban Consulting
- title: (none) -> 4 Channel Optocoupled Input with Schmitt Trigger Module
Changed lines of the file:
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@@
 (kicad_sch (version 20211123) (generator eeschema)
   (paper "A4")
+  (title_block
+    (title "4 Channel Optocoupled Input with Schmitt Trigger Module")
+    (date "2022-04-17")
+    (rev "V1.2")
+    (company "Torban Consulting")
+    (comment 1 "Torban Peterson")
+    (comment 2 "Cameron Eccleston")
+  )
   (junction (at 129.54 100.33) (diameter 0) (color 0 0 0 0)
   )
@@
   )
   (junction (at 129.54 96.52) (diameter 0) (color 0 0 0 0)
-  )
-  (junction (at 129.54 102.87) (diameter 0) (color 0 0 0 0)
   )
   (junction (at 132.08 85.09) (diameter 0) (color 0 0 0 0)
@@
     (stroke (width 0) (type default) (color 0 0 0 0))
   )
-  (wire (pts (xy 128.27 102.87) (xy 129.54 102.87))
-    (stroke (width 0) (type default) (color 0 0 0 0))
-  )
   (wire (pts (xy 100.33 81.28) (xy 100.33 96.52))
     (stroke (width 0) (type default) (color 0 0 0 0))
@@
     (property "Reference" "U1" (id 0) (at 119.38 78.74 0))
     (property "Value" "LTV-847S" (id 1) (at 119.38 81.28 0))
-    (property "Footprint" "Package_SO:SOP-16_4.4x10.4mm_P1.27mm" (id 2) (at 119.38 95.25 0)
+    (property "Footprint" "Package_DIP:SMDIP-16_W9.53mm" (id 2) (at 119.38 95.25 0)
       (effects (font (size 1.27 1.27)) hide)
     )
@@
     (property "Reference" "U2" (id 0) (at 158.75 152.4 0))
     (property "Value" "74HC7014" (id 1) (at 158.75 154.94 0))
-    (property "Footprint" "Package_SO:TSSOP-14_4.4x5mm_P0.65mm" (id 2) (at 158.75 161.29 0)
+    (property "Footprint" "Package_SO:SO-14_3.9x8.65mm_P1.27mm" (id 2) (at 158.75 161.29 0)
       (effects (font (size 1.27 1.27)) hide)
     )
@@
       (effects (font (size 1.27 1.27)) (justify left))
     )
-    (property "Footprint" "Package_SO:TSSOP-14_4.4x5mm_P0.65mm" (id 2) (at 138.43 154.94 0)
+    (property "Footprint" "Package_SO:SO-14_3.9x8.65mm_P1.27mm" (id 2) (at 138.43 154.94 0)
       (effects (font (size 1.27 1.27)) hide)
     )
@@
     (property "Reference" "U2" (id 0) (at 156.21 76.2 0))
     (property "Value" "74HC7014" (id 1) (at 156.21 78.74 0))
-    (property "Footprint" "Package_SO:TSSOP-14_4.4x5mm_P0.65mm" (id 2) (at 156.21 85.09 0)
+    (property "Footprint" "Package_SO:SO-14_3.9x8.65mm_P1.27mm" (id 2) (at 156.21 85.09 0)
       (effects (font (size 1.27 1.27)) hide)
     )
@@
     (property "Reference" "U2" (id 0) (at 156.21 48.26 0))
     (property "Value" "74HC7014" (id 1) (at 156.21 50.8 0))
-    (property "Footprint" "Package_SO:TSSOP-14_4.4x5mm_P0.65mm" (id 2) (at 156.21 57.15 0)
+    (property "Footprint" "Package_SO:SO-14_3.9x8.65mm_P1.27mm" (id 2) (at 156.21 57.15 0)
       (effects (font (size 1.27 1.27)) hide)
     )
@@
     (property "Reference" "U1" (id 0) (at 119.38 50.8 0))
     (property "Value" "LTV-847S" (id 1) (at 119.38 53.34 0))
-    (property "Footprint" "Package_SO:SOP-16_4.4x10.4mm_P1.27mm" (id 2) (at 119.38 67.31 0)
+    (property "Footprint" "Package_DIP:SMDIP-16_W9.53mm" (id 2) (at 119.38 67.31 0)
       (effects (font (size 1.27 1.27)) hide)
     )
@@
     (property "Reference" "U2" (id 0) (at 156.21 34.29 0))
     (property "Value" "74HC7014" (id 1) (at 156.21 36.83 0))
-    (property "Footprint" "Package_SO:TSSOP-14_4.4x5mm_P0.65mm" (id 2) (at 156.21 43.18 0)
+    (property "Footprint" "Package_SO:SO-14_3.9x8.65mm_P1.27mm" (id 2) (at 156.21 43.18 0)
       (effects (font (size 1.27 1.27)) hide)
     )
@@
     (property "Reference" "U2" (id 0) (at 158.75 139.7 0))
     (property "Value" "74HC7014" (id 1) (at 158.75 142.24 0))
-    (property "Footprint" "Package_SO:TSSOP-14_4.4x5mm_P0.65mm" (id 2) (at 158.75 148.59 0)
+    (property "Footprint" "Package_SO:SO-14_3.9x8.65mm_P1.27mm" (id 2) (at 158.75 148.59 0)
       (effects (font (size 1.27 1.27)) hide)
     )
@@
     (property "Reference" "U1" (id 0) (at 119.38 64.77 0))
     (property "Value" "LTV-847S" (id 1) (at 119.38 67.31 0))
-    (property "Footprint" "Package_SO:SOP-16_4.4x10.4mm_P1.27mm" (id 2) (at 119.38 81.28 0)
+    (property "Footprint" "Package_DIP:SMDIP-16_W9.53mm" (id 2) (at 119.38 81.28 0)
       (effects (font (size 1.27 1.27)) hide)
     )
@@
     (property "Reference" "U2" (id 0) (at 156.21 62.23 0))
     (property "Value" "74HC7014" (id 1) (at 156.21 64.77 0))
-    (property "Footprint" "Package_SO:TSSOP-14_4.4x5mm_P0.65mm" (id 2) (at 156.21 71.12 0)
+    (property "Footprint" "Package_SO:SO-14_3.9x8.65mm_P1.27mm" (id 2) (at 156.21 71.12 0)
       (effects (font (size 1.27 1.27)) hide)
     )
@@
     (property "Reference" "U1" (id 0) (at 119.38 36.83 0))
     (property "Value" "LTV-847S" (id 1) (at 119.38 39.37 0))
-    (property "Footprint" "Package_SO:SOP-16_4.4x10.4mm_P1.27mm" (id 2) (at 119.38 53.34 0)
+    (property "Footprint" "Package_DIP:SMDIP-16_W9.53mm" (id 2) (at 119.38 53.34 0)
       (effects (font (size 1.27 1.27)) hide)
     )
@@
     )
     (path "/ed92ba08-98ec-48df-9584-41c899a43f78"
-      (reference "U1") (unit 1) (value "LTV-847S") (footprint "Package_SO:SOP-16_4.4x10.4mm_P1.27mm")
+      (reference "U1") (unit 1) (value "LTV-847S") (footprint "Package_DIP:SMDIP-16_W9.53mm")
     )
     (path "/a6d1221a-1077-412d-8a73-7025f9b4ca20"
-      (reference "U1") (unit 2) (value "LTV-847S") (footprint "Package_SO:SOP-16_4.4x10.4mm_P1.27mm")
+      (reference "U1") (unit 2) (value "LTV-847S") (footprint "Package_DIP:SMDIP-16_W9.53mm")
     )
     (path "/cac6ef5d-79dc-46ad-ba83-77cb1377c287"
-      (reference "U1") (unit 3) (value "LTV-847S") (footprint "Package_SO:SOP-16_4.4x10.4mm_P1.27mm")
+      (reference "U1") (unit 3) (value "LTV-847S") (footprint "Package_DIP:SMDIP-16_W9.53mm")
     )
     (path "/45fc93ca-f8ba-48a8-9189-1c9886475cd3"
-      (reference "U1") (unit 4) (value "LTV-847S") (footprint "Package_SO:SOP-16_4.4x10.4mm_P1.27mm")
+      (reference "U1") (unit 4) (value "LTV-847S") (footprint "Package_DIP:SMDIP-16_W9.53mm")
     )
     (path "/adfaccc9-bb80-495a-9038-d58935037d76"
-      (reference "U2") (unit 1) (value "74HC7014") (footprint "Package_SO:TSSOP-14_4.4x5mm_P0.65mm")
+      (reference "U2") (unit 1) (value "74HC7014") (footprint "Package_SO:SO-14_3.9x8.65mm_P1.27mm")
     )
     (path "/7eebb937-5634-42da-bd7e-2e0260369d0e"
-      (reference "U2") (unit 2) (value "74HC7014") (footprint "Package_SO:TSSOP-14_4.4x5mm_P0.65mm")
+      (reference "U2") (unit 2) (value "74HC7014") (footprint "Package_SO:SO-14_3.9x8.65mm_P1.27mm")
     )
     (path "/d92cfbfa-da4b-4f63-8ad6-7bb6977d4f44"
-      (reference "U2") (unit 3) (value "74HC7014") (footprint "Package_SO:TSSOP-14_4.4x5mm_P0.65mm")
+      (reference "U2") (unit 3) (value "74HC7014") (footprint "Package_SO:SO-14_3.9x8.65mm_P1.27mm")
     )
     (path "/60ca4740-3009-4486-93d6-c2502818122b"
-      (reference "U2") (unit 4) (value "74HC7014") (footprint "Package_SO:TSSOP-14_4.4x5mm_P0.65mm")
+      (reference "U2") (unit 4) (value "74HC7014") (footprint "Package_SO:SO-14_3.9x8.65mm_P1.27mm")
     )
     (path "/bdbfc897-0a76-4ef8-acff-58a8a30c7547"
-      (reference "U2") (unit 5) (value "74HC7014") (footprint "Package_SO:TSSOP-14_4.4x5mm_P0.65mm")
+      (reference "U2") (unit 5) (value "74HC7014") (footprint "Package_SO:SO-14_3.9x8.65mm_P1.27mm")
     )
     (path "/494a6b97-f33e-4834-b724-0c3a3ff54317"
-      (reference "U2") (unit 6) (value "74HC7014") (footprint "Package_SO:TSSOP-14_4.4x5mm_P0.65mm")
+      (reference "U2") (unit 6) (value "74HC7014") (footprint "Package_SO:SO-14_3.9x8.65mm_P1.27mm")
     )
     (path "/49956dd5-35c0-4b9f-8b2a-6f2b8918bd8c"
-      (reference "U2") (unit 7) (value "74HC7014") (footprint "Package_SO:TSSOP-14_4.4x5mm_P0.65mm")
-    )
-  )
+      (reference "U2") (unit 7) (value "74HC7014") (footprint "Package_SO:SO-14_3.9x8.65mm_P1.27mm")
+    )
+  )

Commit message: Random changes
Other:
- moved on the sheet: C2, C3, C4, C5, J1, J2, J5, R1, R10, R11, R12, R2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

Commit message: v2 work
Other:
- moved on the sheet: C2, C3, C4, C5, J1, J2, J5, R1, R10, R11, R12, R2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
